File: hardware/project/ETH1CLCR1/FGEN_Buffer.sch (KiCad schematic (older format))
At the start: 57 parts, among them K1001 9012, K1002 9012, K1003 9012, K1004 9012, Q1001 MMBT4401L, Q1002 MMBT4403L, Q1003 BC847W, Q1004 BC847W, Q1005 BC847W, Q1006 BC847W, U1001 TL072, U1002 LT1468, U1003 AQY212GS, U1004 AD5293BRUZ-20

Commit message: PCB layout
Connections:
- net +12VF is gone; now on net +15VF: C1006.1, C1007.1, U1001.8 (V+)
- net -12VF is gone; now on net -15VF: C1008.1, C1009.1, U1001.4 (V-)
Changed lines of the file:
@@
 	6550 6800 6550 6650
-$Comp
-L ETH1CLCR1:-12VF #PWR01026
-U 1 1 5E570823
-P 6550 6650
-F 0 "#PWR01026" H 6550 6500 50  0001 C CNN
-F 1 "-12VF" H 6565 6823 50  0000 C CNN
-F 2 "" H 6550 6650 50  0001 C CNN
-F 3 "" H 6550 6650 50  0001 C CNN
-	1    6550 6650
-	1    0    0    -1
-$EndComp
-$Comp
-L ETH1CLCR1:-12VF #PWR01025
-U 1 1 5E570ACC
-P 6050 6650
-F 0 "#PWR01025" H 6050 6500 50  0001 C CNN
-F 1 "-12VF" H 6065 6823 50  0000 C CNN
-F 2 "" H 6050 6650 50  0001 C CNN
-F 3 "" H 6050 6650 50  0001 C CNN
-	1    6050 6650
-	1    0    0    -1
-$EndComp
-$Comp
-L ETH1CLCR1:+12VF #PWR01024
-U 1 1 5E5712DC
-P 5550 6650
-F 0 "#PWR01024" H 5550 6500 50  0001 C CNN
-F 1 "+12VF" H 5565 6823 50  0000 C CNN
-F 2 "" H 5550 6650 50  0001 C CNN
-F 3 "" H 5550 6650 50  0001 C CNN
-	1    5550 6650
-	1    0    0    -1
-$EndComp
-$Comp
-L ETH1CLCR1:+12VF #PWR01023
-U 1 1 5E5716B1
-P 5050 6650
-F 0 "#PWR01023" H 5050 6500 50  0001 C CNN
-F 1 "+12VF" H 5065 6823 50  0000 C CNN
-F 2 "" H 5050 6650 50  0001 C CNN
-F 3 "" H 5050 6650 50  0001 C CNN
-	1    5050 6650
-	1    0    0    -1
-$EndComp
-$Comp
-L ETH1CLCR1:+12VF #PWR01022
-U 1 1 5E5719C0
-P 4500 6650
-F 0 "#PWR01022" H 4500 6500 50  0001 C CNN
-F 1 "+12VF" H 4515 6823 50  0000 C CNN
-F 2 "" H 4500 6650 50  0001 C CNN
-F 3 "" H 4500 6650 50  0001 C CNN
-	1    4500 6650
-	1    0    0    -1
-$EndComp
-$Comp
-L ETH1CLCR1:-12VF #PWR01027
-U 1 1 5E571D8E
-P 4500 7250
-F 0 "#PWR01027" H 4500 7100 50  0001 C CNN
-F 1 "-12VF" H 4515 7423 50  0000 C CNN
-F 2 "" H 4500 7250 50  0001 C CNN
-F 3 "" H 4500 7250 50  0001 C CNN
-	1    4500 7250
-	-1   0    0    1
-$EndComp
 $Comp
 L Device:R_POT_TRIM RV1001
@@
 Wire Wire Line
 	2950 6350 2950 6300
+$Comp
+L ETH1CLCR1:+15VF #PWR0107
+U 1 1 5E249D54
+P 4500 6650
+F 0 "#PWR0107" H 4500 6500 50  0001 C CNN
+F 1 "+15VF" H 4515 6823 50  0000 C CNN
+F 2 "" H 4500 6650 50  0001 C CNN
+F 3 "" H 4500 6650 50  0001 C CNN
+	1    4500 6650
+	1    0    0    -1
+$EndComp
+$Comp
+L ETH1CLCR1:+15VF #PWR0108
+U 1 1 5E24CFCD
+P 5050 6650
+F 0 "#PWR0108" H 5050 6500 50  0001 C CNN
+F 1 "+15VF" H 5065 6823 50  0000 C CNN
+F 2 "" H 5050 6650 50  0001 C CNN
+F 3 "" H 5050 6650 50  0001 C CNN
+	1    5050 6650
+	1    0    0    -1
+$EndComp
+$Comp
+L ETH1CLCR1:+15VF #PWR0109
+U 1 1 5E24D5CA
+P 5550 6650
+F 0 "#PWR0109" H 5550 6500 50  0001 C CNN
+F 1 "+15VF" H 5565 6823 50  0000 C CNN
+F 2 "" H 5550 6650 50  0001 C CNN
+F 3 "" H 5550 6650 50  0001 C CNN
+	1    5550 6650
+	1    0    0    -1
+$EndComp
+$Comp
+L ETH1CLCR1:-15VF #PWR0110
+U 1 1 5E24DDD6
+P 6050 6650
+F 0 "#PWR0110" H 6050 6500 50  0001 C CNN
+F 1 "-15VF" H 6065 6823 50  0000 C CNN
+F 2 "" H 6050 6650 50  0001 C CNN
+F 3 "" H 6050 6650 50  0001 C CNN
+	1    6050 6650
+	1    0    0    -1
+$EndComp
+$Comp
+L ETH1CLCR1:-15VF #PWR0111
+U 1 1 5E250E58
+P 6550 6650
+F 0 "#PWR0111" H 6550 6500 50  0001 C CNN
+F 1 "-15VF" H 6565 6823 50  0000 C CNN
+F 2 "" H 6550 6650 50  0001 C CNN
+F 3 "" H 6550 6650 50  0001 C CNN
+	1    6550 6650
+	1    0    0    -1
+$EndComp
+$Comp
+L ETH1CLCR1:-15VF #PWR0112
+U 1 1 5E251502
+P 4500 7250
+F 0 "#PWR0112" H 4500 7100 50  0001 C CNN
+F 1 "-15VF" H 4515 7423 50  0000 C CNN
+F 2 "" H 4500 7250 50  0001 C CNN
+F 3 "" H 4500 7250 50  0001 C CNN
+	1    4500 7250
+	-1   0    0    1
+$EndComp
 $EndSCHEMATC
