File: hardware/project/ETH1CLCR1/FGEN.sch (KiCad schematic (older format))
At the start: 105 parts, among them U901 AD5453YRMZ, U902 LT1468, U903 DG419LDY, U904 LT1468, U905 AD9835, U906 ECS-3225SMV-500-GP-TR, U907 74AHCT1G08, U908 TXB0104D, U909 REF192, U910 TL072, U911 DG408DY, U912 TL072, U913 ADS7818, U914 AD5689BRUZ, U915 TL072

Commit message: Schematic design
Parts:
- U912, U915: footprint (none) -> Package_SO:SOIC-8_3.9x4.9mm_P1.27mm
Changed lines of the file:
@@
 F 0 "U912" H 9600 6800 50  0000 C CNN
 F 1 "TL072" H 9600 6700 50  0000 C CNN
-F 2 "" H 9500 6550 50  0001 C CNN
+F 2 "Package_SO:SOIC-8_3.9x4.9mm_P1.27mm" H 9500 6550 50  0001 C CNN
 F 3 "http://www.ti.com/lit/ds/symlink/tl071.pdf" H 9500 6550 50  0001 C CNN
 	1    9500 6550
@@
 F 0 "U912" H 5450 7150 50  0000 C CNN
 F 1 "TL072" H 5450 7050 50  0000 C CNN
-F 2 "" H 5350 6900 50  0001 C CNN
+F 2 "Package_SO:SOIC-8_3.9x4.9mm_P1.27mm" H 5350 6900 50  0001 C CNN
 F 3 "http://www.ti.com/lit/ds/symlink/tl071.pdf" H 5350 6900 50  0001 C CNN
 	2    5350 6900
@@
 F 0 "U915" H 10300 10150 50  0000 C CNN
 F 1 "TL072" H 10300 10050 50  0000 C CNN
-F 2 "" H 10150 10100 50  0001 C CNN
+F 2 "Package_SO:SOIC-8_3.9x4.9mm_P1.27mm" H 10150 10100 50  0001 C CNN
 F 3 "http://www.ti.com/lit/ds/symlink/tl071.pdf" H 10150 10100 50  0001 C CNN
 	3    10150 10100

Commit message: Schematic design
Parts:
- removed U908: TXB0104D, Package_SO:SOIC-14_3.9x8.7mm_P1.27mm, symbol Logic_LevelTranslator:TXB0104D
- added R801: 10k, Resistor_SMD:R_0603_1608Metric_Pad1.05x0.95mm_HandSolder, symbol Device:R
- added U802, U803: TXB0104PW, Package_SO:TSSOP-14_4.4x5mm_P0.65mm, symbol Logic_LevelTranslator:TXB0104PW
Connections:
- net labels added: +3.3VF, MEAS_CLK, MEAS_CONV, MEAS_DATA
- net labels removed: +3.3VP
- wire segments 371 -> 386
- no-connect marks 13 -> 15
Other:
- moved on the sheet: C918, C919, C920, C921, C922, C923, C924, C927, C928, R912, R918, R919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

Commit message: Need to redesign the AC source, the LT1468 is too slow.
Parts:
- added R802, R803: 10k, Resistor_SMD:R_0603_1608Metric_Pad1.05x0.95mm_HandSolder, symbol Device:R
- added U804: LT1468, Package_SO:SSOP-8_3.9x5.05mm_P1.27mm, symbol ETH1CLCR1:LT1468
- R901, R907: value R -> 10k
- R904: value R -> 200k
- R934, R940: value R -> NC
- R938: value R -> 0
Connections:
- net +15VF: now also U804.7 (V+)
- net -15VF: now also U804.4 (V-)
- net AGNDF: now also U804.3 (+)
- net at C901.2, R904.2, R907.1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: no longer R901.1
- net at C901.1, R904.1, U904.6: now also R803.2; no longer U903.1
- new net: R802.2, R803.1, R901.1, U804.2 (-)
- new net: R802.1, U804.6, U903.1
- no-connect marks 15 -> 17
Other:
- moved on the sheet: C901, C902, C903, C908, C918, C919, C920, C921, C922, C923, C924, C927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

Commit message: Footprint asigment (not finished).
Parts:
- C815: renamed from C915; footprint Capacitor_SMD:C_0603_1608Metric_Pad1.05x0.95mm_HandSolder -> Capacitor_SMD:C_0805_2012Metric_Pad1.15x1.40mm_HandSolder
- R803: renamed from R904; value 200k -> 10k
- R804: renamed from R901; value 10k -> 1k
- R805: renamed from R802; value 10k -> 1k
- R808: renamed from R907; value 10k -> 1k
- R809: renamed from R803; value 10k -> 1k
- renumbered C901 to C801, C902 to C802, C903 to C803, C904 to C804, C905 to C805, C906 to C806, C907 to C807, C908 to C808, C909 to C809, C910 to C810, C911 to C811, C912 to C812, C913 to C813, C914 to C814, C916 to C816, C917 to C817, C918 to C818, C919 to C819, C920 to C820, C921 to C821, C922 to C822, C923 to C823, C924 to C824, C925 to C825, C926 to C826, C927 to C827, C928 to C828, C929 to C829, C930 to C830, C931 to C831, C932 to C832, C933 to C833, C934 to C834, C935 to C835, C936 to C836, C937 to C837, C938 to C838, C939 to C839, C940 to C840, C941 to C841, C942 to C842, C943 to C843, D901 to D801, L901 to L801, L902 to L802, L903 to L803, R902 to R801, R903 to R802, R905 to R806, R906 to R807, R908 to R810, R909 to R811, R910 to R812, R911 to R813, R912 to R814, R913 to R815, R914 to R816, R915 to R817, R916 to R818, R917 to R819, R918 to R820, R919 to R821, R920 to R822, R921 to R823, R922 to R824, R923 to R825, R924 to R826, R925 to R827, R926 to R828, R927 to R829, R928 to R830, R929 to R831, R930 to R832, R931 to R833, R932 to R834, R933 to R835, R934 to R836, R935 to R837, R936 to R838, R937 to R839, R938 to R840, R939 to R841, R801 to R842, R940 to R843, R941 to R844, R942 to R845, R943 to R846, U901 to U801, U902 to U802, U904 to U803, U903 to U804, U905 to U805, U804 to U806, U906 to U807, U907 to U808, U802 to U809, U909 to U810, U910 to U811, U911 to U812, U912 to U813, U913 to U814, U914 to U815, U803 to U816, U915 to U817

Commit message: Modification in schematic and PCB layout.
Parts:
- C815: footprint Capacitor_SMD:C_0805_2012Metric_Pad1.15x1.40mm_HandSolder -> Capacitor_SMD:C_0603_1608Metric_Pad1.05x0.95mm_HandSolder
Changed lines of the file:
@@
 F 0 "C815" H 2115 5196 50  0000 L CNN
 F 1 "1u" H 2115 5105 50  0000 L CNN
-F 2 "Capacitor_SMD:C_0805_2012Metric_Pad1.15x1.40mm_HandSolder" H 2038 5000 50  0001 C CNN
+F 2 "Capacitor_SMD:C_0603_1608Metric_Pad1.05x0.95mm_HandSolder" H 2038 5000 50  0001 C CNN
 F 3 "~" H 2000 5150 50  0001 C CNN
 	1    2000 5150

Commit message: PCB layout
Parts:
- removed C802, C820: 1n, Capacitor_SMD:C_0603_1608Metric_Pad1.05x0.95mm_HandSolder, symbol Device:C
- removed C818, C827, C834: 100n, Capacitor_SMD:C_0603_1608Metric_Pad1.05x0.95mm_HandSolder, symbol Device:C
- removed C819: 220p, Capacitor_SMD:C_0603_1608Metric_Pad1.05x0.95mm_HandSolder, symbol Device:C
- removed C821: 470p, Capacitor_SMD:C_0603_1608Metric_Pad1.05x0.95mm_HandSolder, symbol Device:C
- removed C822: 330p, Capacitor_SMD:C_0603_1608Metric_Pad1.05x0.95mm_HandSolder, symbol Device:C
- removed C823: 150p, Capacitor_SMD:C_0603_1608Metric_Pad1.05x0.95mm_HandSolder, symbol Device:C
- removed C824: 4n7, Capacitor_SMD:C_0603_1608Metric_Pad1.05x0.95mm_HandSolder, symbol Device:C
- removed C828: 2u2, Capacitor_SMD:C_0805_2012Metric_Pad1.15x1.40mm_HandSolder, symbol Device:C
- removed R814, R820, R821, R824, R826, R833, R834, R835, R837, R841, R842, R845, R846: 10k, Resistor_SMD:R_0603_1608Metric_Pad1.05x0.95mm_HandSolder, symbol Device:R
- removed R825: 619, Resistor_SMD:R_0603_1608Metric_Pad1.05x0.95mm_HandSolder, symbol Device:R
- removed R827, R828, R829: 6k81, Resistor_SMD:R_0603_1608Metric_Pad1.05x0.95mm_HandSolder, symbol Device:R
- removed R830: 70k, Resistor_SMD:R_0603_1608Metric_Pad1.05x0.95mm_HandSolder, symbol Device:R
- removed R832: 237k, Resistor_SMD:R_0603_1608Metric_Pad1.05x0.95mm_HandSolder, symbol Device:R
- removed U809, U816: TXB0104PW, Package_SO:TSSOP-14_4.4x5mm_P0.65mm, symbol Logic_LevelTranslator:TXB0104PW
- removed U812: DG408DY, Package_SO:TSSOP-16_4.4x5mm_P0.65mm, symbol ETH1CLCR1:DG408DY
- removed U813, U817: TL072, Package_SO:SOIC-8_3.9x4.9mm_P1.27mm, symbol Amplifier_Operational:TL072
- removed U814: ADS7818, Package_SO:MSOP-8_3x3mm_P0.65mm, symbol ETH1CLCR1:ADS7818
- R827: renamed from R801; value 10k -> R
- U803: renamed from U808; footprint Package_TO_SOT_SMD:SOT-353_SC-70-5_Handsoldering -> Package_TO_SOT_SMD:SOT-353_SC-70-5
- renumbered C829 to C801, C814 to C802, C830 to C803, C831 to C804, C815 to C805, C832 to C806, C833 to C807, C835 to C808, C836 to C809, C816 to C810, C837 to C811, C825 to C812, C817 to C813, C804 to C814, C838 to C815, C813 to C816, C826 to C817, C809 to C818, C805 to C819, C810 to C820, C806 to C821, C839 to C822, C811 to C823, C807 to C824, C840 to C825, C812 to C826, C841 to C827, C808 to C828, C842 to C829, C843 to C830, C803 to C831, C801 to C832, R822 to R801, R840 to R802, R836 to R803, R843 to R804, R823 to R805, R813 to R806, R815 to R807, R816 to R808, R806 to R809, R817 to R810, R818 to R811, R831 to R812, R812 to R813, R838 to R814, R844 to R815, R839 to R816, R810 to R817, R819 to R818, R811 to R819, R807 to R820, R802 to R821, R808 to R822, R803 to R823, R804 to R824, R809 to R825, R805 to R826, U807 to U801, U810 to U802, U815 to U804, U811 to U806, U804 to U807, U801 to U808, U802 to U809, U803 to U810, U806 to U811
Connections:
- net MEAS_OUT is gone; now on net AGNDF: R827.1
- net V_OFFSET: now also U806.7
- net at U806.5 (+): now also C812.1, R812.1
- net at U806.6 (-): now also C817.2, R814.1, R815.1, R816.2; no longer U806.7
- no-connect marks 17 -> 9
Other:
- moved on the sheet: C808, C809, C811, C815, C822, C825, C827, C829, C830, D801C, R827, U806B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
