File: hardware/project/ETH1CLCR1/FGEN.sch (KiCad schematic (older format))
At the start: 81 parts, among them U1401 ECS-3225SMV-500-GP-TR, U1402 REF192, U1403 74AHCT1G08, U1404 AD5689BRUZ, U1405 AD9835, U1406 TL072, U1407 DG419LDY, U1408 AD5453YRMZ, U1409 LT1468, U1410 LT1468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

Commit message: Fixed problem with LT1468 stablity (changed 1p5 to 27p C). AD5453 software works. Changed U1410 gain from 10 to 5.
Parts:
- C1434, C1436: value 1p5 -> 20p
- R1422: value 10k -> DNP
- R1424: value 10k -> 2k
Other:
- note added: "2k4 tmp"
Changed lines of the file:
@@
 P 10150 1700
 F 0 "C1434" H 10265 1746 50  0000 L CNN
-F 1 "1p5" H 10265 1655 50  0000 L CNN
+F 1 "20p" H 10265 1655 50  0000 L CNN
 F 2 "Capacitor_SMD:C_0603_1608Metric_Pad1.05x0.95mm_HandSolder" H 10188 1550 50  0001 C CNN
 F 3 "~" H 10150 1700 50  0001 C CNN
@@
 	1    0    0    -1
 $EndComp
-$Comp
-L Device:R R1423
-U 1 1 5DDFC921
-P 11500 2150
-F 0 "R1423" V 11293 2150 50  0000 C CNN
-F 1 "1k" V 11384 2150 50  0000 C CNN
-F 2 "Resistor_SMD:R_0603_1608Metric_Pad1.05x0.95mm_HandSolder" V 11430 2150 50  0001 C CNN
-F 3 "~" H 11500 2150 50  0001 C CNN
-	1    11500 2150
-	0    1    1    0
-$EndComp
 Wire Wire Line
 	11350 2150 11250 2150
@@
 Wire Wire Line
 	11850 2150 11750 2150
-$Comp
-L Device:R R1424
-U 1 1 5E01472E
-P 12200 1500
-F 0 "R1424" V 11993 1500 50  0000 C CNN
-F 1 "10k" V 12084 1500 50  0000 C CNN
-F 2 "Resistor_SMD:R_0603_1608Metric_Pad1.05x0.95mm_HandSolder" V 12130 1500 50  0001 C CNN
-F 3 "~" H 12200 1500 50  0001 C CNN
-	1    12200 1500
-	0    1    1    0
-$EndComp
 Wire Wire Line
 	12050 1500 11750 1500
@@
 P 12200 1100
 F 0 "C1436" V 11948 1100 50  0000 C CNN
-F 1 "1p5" V 12039 1100 50  0000 C CNN
+F 1 "20p" V 12039 1100 50  0000 C CNN
 F 2 "Capacitor_SMD:C_0603_1608Metric_Pad1.05x0.95mm_HandSolder" H 12238 950 50  0001 C CNN
 F 3 "~" H 12200 1100 50  0001 C CNN
@@
 $EndComp
 $Comp
-L Device:R R1426
-U 1 1 5E35B1C2
-P 13350 2250
-F 0 "R1426" V 13143 2250 50  0000 C CNN
-F 1 "1k" V 13234 2250 50  0000 C CNN
-F 2 "Resistor_SMD:R_0603_1608Metric_Pad1.05x0.95mm_HandSolder" V 13280 2250 50  0001 C CNN
-F 3 "~" H 13350 2250 50  0001 C CNN
-	1    13350 2250
-	0    1    1    0
-$EndComp
-$Comp
 L ETH1CLCR1:+15VF #PWR01482
 U 1 1 5E35B1C8
@@
 P 11500 1100
 F 0 "R1422" V 11293 1100 50  0000 C CNN
-F 1 "10k" V 11384 1100 50  0000 C CNN
+F 1 "DNP" V 11384 1100 50  0000 C CNN
 F 2 "Resistor_SMD:R_0603_1608Metric_Pad1.05x0.95mm_HandSolder" V 11430 1100 50  0001 C CNN
 F 3 "~" H 11500 1100 50  0001 C CNN
@@
 Wire Wire Line
 	1800 2450 1800 2650
+$Comp
+L Device:R R1426
+U 1 1 5E35B1C2
+P 13350 2250
+F 0 "R1426" V 13143 2250 50  0000 C CNN
+F 1 "1k" V 13234 2250 50  0000 C CNN
+F 2 "Resistor_SMD:R_0603_1608Metric_Pad1.05x0.95mm_HandSolder" V 13280 2250 50  0001 C CNN
+F 3 "~" H 13350 2250 50  0001 C CNN
+	1    13350 2250
+	0    1    1    0
+$EndComp
+$Comp
+L Device:R R1424
+U 1 1 5E01472E
+P 12200 1500
+F 0 "R1424" V 11993 1500 50  0000 C CNN
+F 1 "2k" V 12084 1500 50  0000 C CNN
+F 2 "Resistor_SMD:R_0603_1608Metric_Pad1.05x0.95mm_HandSolder" V 12130 1500 50  0001 C CNN
+F 3 "~" H 12200 1500 50  0001 C CNN
+	1    12200 1500
+	0    1    1    0
+$EndComp
+$Comp
+L Device:R R1423
+U 1 1 5DDFC921
+P 11500 2150
+F 0 "R1423" V 11293 2150 50  0000 C CNN
+F 1 "1k" V 11384 2150 50  0000 C CNN
+F 2 "Resistor_SMD:R_0603_1608Metric_Pad1.05x0.95mm_HandSolder" V 11430 2150 50  0001 C CNN
+F 3 "~" H 11500 2150 50  0001 C CNN
+	1    11500 2150
+	0    1    1    0
+$EndComp
+Text Notes 12350 1400 0    50   ~ 0
+2k4 tmp
 $EndSCHEMATC

Commit message: Software development.
Other:
- note added: "5k05 tmp"
- note removed: "2k4 tmp"
Changed lines of the file:
@@
 $EndComp
 Text Notes 12350 1400 0    50   ~ 0
-2k4 tmp
+5k05 tmp
 $EndSCHEMATC
