File: hardware/project/ETH1CLCR1/Isolation.sch (KiCad schematic (older format))
At the start: 3 parts, among them U801 ADuM3151

Commit message: Footprint asigment (not finished).
Parts:
- renumbered C801 to C701, C802 to C702, U801 to U701
Changed lines of the file:
@@
 $EndDescr
 $Comp
-L ETH1CLCR1:ADuM3151 U801
+L ETH1CLCR1:ADuM3151 U701
 U 1 1 5DD9E9B5
 P 5500 2800
-F 0 "U801" H 5500 3665 50  0000 C CNN
+F 0 "U701" H 5500 3665 50  0000 C CNN
 F 1 "ADuM3151" H 5500 3574 50  0000 C CNN
 F 2 "Package_SO:SSOP-20_5.3x7.2mm_P0.65mm" H 7400 3250 50  0001 C CNN
@@
 	4750 2200 4800 2200
 $Comp
-L power:GND #PWR0807
+L power:GND #PWR0707
 U 1 1 5DDA742F
 P 4750 3500
-F 0 "#PWR0807" H 4750 3250 50  0001 C CNN
+F 0 "#PWR0707" H 4750 3250 50  0001 C CNN
 F 1 "GND" H 4755 3327 50  0000 C CNN
 F 2 "" H 4750 3500 50  0001 C CNN
@@
 	5500 3600 5500 7700
 $Comp
-L power:+3.3V #PWR0805
+L power:+3.3V #PWR0705
 U 1 1 5DDAF4AD
 P 4750 2100
-F 0 "#PWR0805" H 4750 1950 50  0001 C CNN
+F 0 "#PWR0705" H 4750 1950 50  0001 C CNN
 F 1 "+3.3V" H 4765 2273 50  0000 C CNN
 F 2 "" H 4750 2100 50  0001 C CNN
@@
 $EndComp
 $Comp
-L ETH1CLCR1:+3.3VF #PWR0806
+L ETH1CLCR1:+3.3VF #PWR0706
 U 1 1 5DDAFA37
 P 6250 2100
-F 0 "#PWR0806" H 6250 1950 50  0001 C CNN
+F 0 "#PWR0706" H 6250 1950 50  0001 C CNN
 F 1 "+3.3VF" H 6265 2273 50  0000 C CNN
 F 2 "" H 6250 2100 50  0001 C CNN
@@
 	6250 2200 6200 2200
 $Comp
-L ETH1CLCR1:DGNDF #PWR0808
+L ETH1CLCR1:DGNDF #PWR0708
 U 1 1 5DDB1D03
 P 6250 3500
-F 0 "#PWR0808" H 6250 3250 50  0001 C CNN
+F 0 "#PWR0708" H 6250 3250 50  0001 C CNN
 F 1 "DGNDF" H 6255 3327 50  0000 C CNN
 F 2 "" H 6250 3500 50  0001 C CNN
@@
 	6250 3400 6250 3300
 $Comp
-L power:+3.3V #PWR0801
+L power:+3.3V #PWR0701
 U 1 1 5DDB5B86
 P 4750 1150
-F 0 "#PWR0801" H 4750 1000 50  0001 C CNN
+F 0 "#PWR0701" H 4750 1000 50  0001 C CNN
 F 1 "+3.3V" H 4765 1323 50  0000 C CNN
 F 2 "" H 4750 1150 50  0001 C CNN
@@
 $EndComp
 $Comp
-L Device:C C801
+L Device:C C701
 U 1 1 5DDB7F1A
 P 4750 1300
-F 0 "C801" H 4865 1346 50  0000 L CNN
+F 0 "C701" H 4865 1346 50  0000 L CNN
 F 1 "100n" H 4865 1255 50  0000 L CNN
 F 2 "Capacitor_SMD:C_0603_1608Metric_Pad1.05x0.95mm_HandSolder" H 4788 1150 50  0001 C CNN
@@
 $EndComp
 $Comp
-L power:GND #PWR0803
+L power:GND #PWR0703
 U 1 1 5DDBBA7D
 P 4750 1450
-F 0 "#PWR0803" H 4750 1200 50  0001 C CNN
+F 0 "#PWR0703" H 4750 1200 50  0001 C CNN
 F 1 "GND" H 4755 1277 50  0000 C CNN
 F 2 "" H 4750 1450 50  0001 C CNN
@@
 $EndComp
 $Comp
-L Device:C C802
+L Device:C C702
 U 1 1 5DDC10CB
 P 6250 1300
-F 0 "C802" H 6365 1346 50  0000 L CNN
+F 0 "C702" H 6365 1346 50  0000 L CNN
 F 1 "100n" H 6365 1255 50  0000 L CNN
 F 2 "Capacitor_SMD:C_0603_1608Metric_Pad1.05x0.95mm_HandSolder" H 6288 1150 50  0001 C CNN
@@
 $EndComp
 $Comp
-L ETH1CLCR1:+3.3VF #PWR0802
+L ETH1CLCR1:+3.3VF #PWR0702
 U 1 1 5DDC1869
 P 6250 1150
-F 0 "#PWR0802" H 6250 1000 50  0001 C CNN
+F 0 "#PWR0702" H 6250 1000 50  0001 C CNN
 F 1 "+3.3VF" H 6265 1323 50  0000 C CNN
 F 2 "" H 6250 1150 50  0001 C CNN
@@
 $EndComp
 $Comp
-L ETH1CLCR1:DGNDF #PWR0804
+L ETH1CLCR1:DGNDF #PWR0704
 U 1 1 5DDC21F1
 P 6250 1450
-F 0 "#PWR0804" H 6250 1200 50  0001 C CNN
+F 0 "#PWR0704" H 6250 1200 50  0001 C CNN
 F 1 "DGNDF" H 6255 1277 50  0000 C CNN
 F 2 "" H 6250 1450 50  0001 C CNN

Commit message: Modification in schematic and PCB layout.
Connections:
- net +3.3VF renamed +3.3VP
Changed lines of the file:
@@
 $Descr A4 11693 8268
 encoding utf-8
-Sheet 9 16
+Sheet 7 16
 Title ""
 Date ""
@@
 Wire Notes Line
 	5500 3600 5500 7700
-$Comp
-L power:+3.3V #PWR0705
-U 1 1 5DDAF4AD
-P 4750 2100
-F 0 "#PWR0705" H 4750 1950 50  0001 C CNN
-F 1 "+3.3V" H 4765 2273 50  0000 C CNN
-F 2 "" H 4750 2100 50  0001 C CNN
-F 3 "" H 4750 2100 50  0001 C CNN
-	1    4750 2100
-	1    0    0    -1
-$EndComp
-$Comp
-L ETH1CLCR1:+3.3VF #PWR0706
-U 1 1 5DDAFA37
-P 6250 2100
-F 0 "#PWR0706" H 6250 1950 50  0001 C CNN
-F 1 "+3.3VF" H 6265 2273 50  0000 C CNN
-F 2 "" H 6250 2100 50  0001 C CNN
-F 3 "" H 6250 2100 50  0001 C CNN
-	1    6250 2100
-	1    0    0    -1
-$EndComp
 Wire Wire Line
 	6250 2100 6250 2200
@@
 	6250 3400 6250 3300
 $Comp
-L power:+3.3V #PWR0701
-U 1 1 5DDB5B86
-P 4750 1150
-F 0 "#PWR0701" H 4750 1000 50  0001 C CNN
-F 1 "+3.3V" H 4765 1323 50  0000 C CNN
-F 2 "" H 4750 1150 50  0001 C CNN
-F 3 "" H 4750 1150 50  0001 C CNN
-	1    4750 1150
-	1    0    0    -1
-$EndComp
-$Comp
 L Device:C C701
 U 1 1 5DDB7F1A
@@
 F 3 "~" H 6250 1300 50  0001 C CNN
 	1    6250 1300
-	1    0    0    -1
-$EndComp
-$Comp
-L ETH1CLCR1:+3.3VF #PWR0702
-U 1 1 5DDC1869
-P 6250 1150
-F 0 "#PWR0702" H 6250 1000 50  0001 C CNN
-F 1 "+3.3VF" H 6265 1323 50  0000 C CNN
-F 2 "" H 6250 1150 50  0001 C CNN
-F 3 "" H 6250 1150 50  0001 C CNN
-	1    6250 1150
 	1    0    0    -1
 $EndComp
@@
 Wire Wire Line
 	6250 2900 6200 2900
+$Comp
+L power:+3.3V #PWR0101
+U 1 1 5E29D877
+P 4750 2100
+F 0 "#PWR0101" H 4750 1950 50  0001 C CNN
+F 1 "+3.3V" H 4765 2273 50  0000 C CNN
+F 2 "" H 4750 2100 50  0001 C CNN
+F 3 "" H 4750 2100 50  0001 C CNN
+	1    4750 2100
+	1    0    0    -1
+$EndComp
+$Comp
+L power:+3.3V #PWR0102
+U 1 1 5E29DD7E
+P 4750 1150
+F 0 "#PWR0102" H 4750 1000 50  0001 C CNN
+F 1 "+3.3V" H 4765 1323 50  0000 C CNN
+F 2 "" H 4750 1150 50  0001 C CNN
+F 3 "" H 4750 1150 50  0001 C CNN
+	1    4750 1150
+	1    0    0    -1
+$EndComp
+$Comp
+L power:+3.3VP #PWR0103
+U 1 1 5E29E93A
+P 6250 2100
+F 0 "#PWR0103" H 6400 2050 50  0001 C CNN
+F 1 "+3.3VP" H 6270 2243 50  0000 C CNN
+F 2 "" H 6250 2100 50  0001 C CNN
+F 3 "" H 6250 2100 50  0001 C CNN
+	1    6250 2100
+	1    0    0    -1
+$EndComp
+$Comp
+L power:+3.3VP #PWR0104
+U 1 1 5E29EC11
+P 6250 1150
+F 0 "#PWR0104" H 6400 1100 50  0001 C CNN
+F 1 "+3.3VP" H 6270 1293 50  0000 C CNN
+F 2 "" H 6250 1150 50  0001 C CNN
+F 3 "" H 6250 1150 50  0001 C CNN
+	1    6250 1150
+	1    0    0    -1
+$EndComp
 $EndSCHEMATC
