File: hardware/project/ETH1CLCR1/DAC.sch (KiCad schematic (older format))
At the start: 57 parts, among them U1501 TL074, U1502 REF192, U1503 DAC7564, U1504 TL074, U1505 DAC7564

Commit message: Footprint asigment (not finished).
Parts:
- removed C1514, C1525, C1526: 100n, Capacitor_SMD:C_0603_1608Metric_Pad1.05x0.95mm_HandSolder, symbol Device:C
- removed U1503, U1505: DAC7564, symbol ETH1CLCR1:DAC7564
- added U1404: DAC7568ICPWR, Package_SO:TSSOP-16_4.4x5mm_P0.65mm, symbol ETH1CLCR1:DAC7568ICPWR
- C1406: renamed from C1505; footprint Capacitor_SMD:C_0603_1608Metric_Pad1.05x0.95mm_HandSolder -> Capacitor_SMD:C_0805_2012Metric_Pad1.15x1.40mm_HandSolder
- U1401: renamed from U1501; footprint (none) -> Package_SO:SOIC-14_3.9x8.7mm_P1.27mm
- U1402: renamed from U1504; footprint (none) -> Package_SO:SOIC-14_3.9x8.7mm_P1.27mm
- renumbered C1501 to C1401, C1515 to C1402, C1502 to C1403, C1517 to C1404, C1503 to C1405, C1507 to C1407, C1516 to C1408, C1510 to C1409, C1518 to C1410, C1508 to C1411, C1519 to C1412, C1511 to C1413, C1521 to C1414, C1509 to C1415, C1512 to C1416, C1504 to C1417, C1506 to C1418, C1513 to C1419, C1523 to C1420, C1524 to C1421, R1501 to R1401, R1517 to R1402, R1502 to R1403, R1504 to R1404, R1519 to R1405, R1523 to R1406, R1503 to R1407, R1520 to R1408, R1505 to R1409, R1518 to R1410, R1508 to R1411, R1514 to R1412, R1521 to R1413, R1524 to R1414, R1509 to R1415, R1522 to R1416, R1506 to R1417, R1525 to R1418, R1510 to R1419, R1515 to R1420, R1527 to R1421, R1531 to R1422, R1511 to R1423, R1528 to R1424, R1507 to R1425, R1512 to R1426, R1516 to R1427, R1513 to R1428, U1502 to U1403
Connections:
- net labels added: DAC_ADC_OFFS1, DAC_ADC_OFFS2, DAC_PA_OFFS1, DAC_PA_OFFS2, DAC_PA_OFFS3, DAC_PA_OFFS4, DAC_RR_OFFS1, DAC_~CLR, DAC_~LDAC
- net labels removed: DAC1_LDAC, DAC1_~ENABLE, DAC2_LDAC, DAC2_~ENABLE, DGNDF
- wire segments 218 -> 198
Other:
- moved on the sheet: C1401, C1403, C1405, C1406, C1407, C1409, C1411, C1413, C1415, C1416, C1420, C1421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

Commit message: PCB layout
Parts:
- C1406: footprint Capacitor_SMD:C_0805_2012Metric_Pad1.15x1.40mm_HandSolder -> Capacitor_SMD:C_0603_1608Metric_Pad1.05x0.95mm_HandSolder
Other:
- moved on the sheet: C1405
Changed lines of the file:
@@
 	2950 2600 2950 2550
 Wire Wire Line
-	2950 2550 2300 2550
+	2950 2550 2200 2550
 Wire Wire Line
-	2300 2550 2300 2900
+	2200 2550 2200 2900
 Wire Wire Line
-	2300 2900 2550 2900
+	2200 2900 2550 2900
 Connection ~ 2950 2550
 Wire Wire Line
@@
 L Device:C C?
 U 1 1 5E3772F7
-P 2300 3100
+P 2200 3100
 AR Path="/5DEEF70B/5E3772F7" Ref="C?"  Part="1"
 AR Path="/5E087FDC/5E3772F7" Ref="C1405"  Part="1"
-F 0 "C1405" H 2415 3146 50  0000 L CNN
-F 1 "10u" H 2415 3055 50  0000 L CNN
-F 2 "Capacitor_SMD:C_0805_2012Metric_Pad1.15x1.40mm_HandSolder" H 2338 2950 50  0001 C CNN
-F 3 "~" H 2300 3100 50  0001 C CNN
-	1    2300 3100
+F 0 "C1405" H 2315 3146 50  0000 L CNN
+F 1 "10u" H 2315 3055 50  0000 L CNN
+F 2 "Capacitor_SMD:C_0805_2012Metric_Pad1.15x1.40mm_HandSolder" H 2238 2950 50  0001 C CNN
+F 3 "~" H 2200 3100 50  0001 C CNN
+	1    2200 3100
 	1    0    0    -1
 $EndComp
 Wire Wire Line
-	2300 2950 2300 2900
-Connection ~ 2300 2900
+	2200 2950 2200 2900
+Connection ~ 2200 2900
 Wire Wire Line
-	2300 3250 2300 3300
+	2200 3250 2200 3300
 Wire Wire Line
-	2300 3300 2950 3300
+	2200 3300 2950 3300
 Wire Wire Line
 	2950 3300 2950 3200
@@
 F 0 "C1406" H 3465 3146 50  0000 L CNN
 F 1 "1u" H 3465 3055 50  0000 L CNN
-F 2 "Capacitor_SMD:C_0805_2012Metric_Pad1.15x1.40mm_HandSolder" H 3388 2950 50  0001 C CNN
+F 2 "Capacitor_SMD:C_0603_1608Metric_Pad1.05x0.95mm_HandSolder" H 3388 2950 50  0001 C CNN
 F 3 "~" H 3350 3100 50  0001 C CNN
 	1    3350 3100

Commit message: Redesinged ADC schematic.
Parts:
- renumbered C1405 to C1401, C1417 to C1402, C1418 to C1403, C1406 to C1404, C1419 to C1405, C1420 to C1406, C1421 to C1407, C1401 to C1408, C1407 to C1409, C1411 to C1410, C1415 to C1411, C1403 to C1412, C1409 to C1413, C1413 to C1414, C1416 to C1415, C1402 to C1416, C1408 to C1417, C1412 to C1418, C1404 to C1419, C1410 to C1420, C1414 to C1421, R1409 to R1402, R1417 to R1403, R1425 to R1404, R1403 to R1405, R1407 to R1406, R1411 to R1407, R1415 to R1408, R1419 to R1409, R1423 to R1410, R1426 to R1411, R1428 to R1412, R1404 to R1413, R1412 to R1414, R1420 to R1415, R1427 to R1416, R1402 to R1417, R1410 to R1418, R1418 to R1419, R1405 to R1420, R1408 to R1421, R1413 to R1422, R1416 to R1423, R1421 to R1424, R1424 to R1425, R1406 to R1426, R1414 to R1427, R1422 to R1428

Commit message: Redesigned the power supply, added humidy+temp. sensor.
Parts:
- renumbered C1401 to C1001, C1402 to C1002, C1403 to C1003, C1404 to C1004, C1405 to C1005, C1406 to C1006, C1407 to C1007, C1408 to C1008, C1409 to C1009, C1410 to C1010, C1411 to C1011, C1412 to C1012, C1413 to C1013, C1414 to C1014, C1415 to C1015, C1416 to C1016, C1417 to C1017, C1418 to C1018, C1419 to C1019, C1420 to C1020, C1421 to C1021, R1401 to R1001, R1402 to R1002, R1403 to R1003, R1404 to R1004, R1405 to R1005, R1406 to R1006, R1407 to R1007, R1408 to R1008, R1409 to R1009, R1410 to R1010, R1411 to R1011, R1412 to R1012, R1413 to R1013, R1414 to R1014, R1415 to R1015, R1416 to R1016, R1417 to R1017, R1418 to R1018, R1419 to R1019, R1420 to R1020, R1421 to R1021, R1422 to R1022, R1423 to R1023, R1424 to R1024, R1425 to R1025, R1426 to R1026, R1427 to R1027, R1428 to R1028, U1401 to U1001, U1402 to U1002, U1403 to U1003, U1404 to U1004

Commit message: Changes in schematics.
Parts:
- added C1001, C1006: 100n, Capacitor_SMD:C_0603_1608Metric_Pad1.05x0.95mm_HandSolder, symbol Device:C
- added C1008: 1u, Capacitor_SMD:C_0603_1608Metric_Pad1.05x0.95mm_HandSolder, symbol Device:C
- U1004: value DAC7568ICPWR -> DAC8568IBPWR; symbol ETH1CLCR1:DAC7568ICPWR -> ETH1CLCR1:DAC8568IxPWR
- renumbered C1001 to C1002, C1002 to C1003, C1003 to C1005, C1005 to C1007, C1006 to C1009, C1007 to C1010, C1008 to C1011, C1009 to C1012, C1010 to C1013, C1011 to C1014, C1012 to C1015, C1013 to C1016, C1014 to C1017, C1015 to C1018, C1016 to C1019, C1017 to C1020, C1018 to C1021, C1019 to C1022, C1020 to C1023, C1021 to C1024
Connections:
- net +2V5REF: now also C1006.1
- net +3.3VF: now also C1008.1
- net +5VF: now also C1001.1
- net AGNDF: now also C1001.2, C1006.2, C1008.2
Other:
- note added: "NOTE: DAC shout rest to midlescale of the V ref. By startup it will set the outputs of the TL074 op amps to 0V."
- moved on the sheet: C1002, C1004, C1009, C1010, U1003
