File: hardware/project/ETH1CLCR1/ETH1CLCR1.kicad_pcb (KiCad board)
At the start: 6 copper layers, 160 x 100 mm, 671 parts, among them J1201 C64AC, J1301 Conn_02x05, J301 Conn_02x01, J302 Conn_02x05, J601 Conn_02x05, K1201 HE3621A0510, K1202 HE3621A0510, K1203 HE3621A0510, K1204 HE3621A0510, K1205 HE3621A0510, K1206 HE3621A0510, K701 9012, K702 9012, K703 9012, K704 9012, K801 TQ2SA-5V, Q1101 BC847, Q1102 BC847, Q1103 BC847, Q1104 BC847, Q501 IRFR5410, Q701 BC847W, Q702 BC847W, Q703 BC847W, Q704 BC847W, Q705 MMBT4401L, Q706 MMBT4403L, Q801 BC847W, Q802 2N2218A, Q803 2N2904A, Q804 BC847W, U1001 TL074, U1002 TL074, U1003 REF192, U1004 DAC7568ICPWR, U1101 ADG419BR, U1102 ADG419BR, U1103 AD8606-2-MSOP, U1104 AD7380, U1105 AD8605, U1106 AD8605, U1107 LT6350, U1108 LT6350, U1109 OPA602, U1110 OPA602, U1111 PGA103, U1112 PGA103, U1201 ULN2003A, U1301 24LC08B-E/MS, U1302 STM32H743ZI, U1401 ECS-3225SMV-500-GP-TR, U1402 REF192, U1403 74AHCT1G08, U1404 AD5689BRUZ, U1405 AD9835, U1406 TL072, U1407 DG419LDY, U1408 AD5453YRMZ, U1409 LT1468, U1410 LT1468, U1411 LT1468, U1501 LT8330_S6, U1502 LT8330_S6, U1503 MC7815BD2TG, U1504 MC7915BD2TG, U1505 MC78M12ABDTRKG, U1506 MC79M12CDTG, U1507 TSR2-2450, U1508 TSR1-2490, U1509 LM1117IMP-3.3/NOPB, U1510 LM1117IMP-3.3/NOPB, U1511 LM1117IMP-5.0/NOPB, U201 LAN8742A, U202 LC03-3.3, U203 LC03-3.3, U301 STM32F765ZGT6, U302 24LC08B-E/MS, U303 HDC1080, U401 TXB0104PW, U402 ADuM5402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

Commit message: Changes in schematics.
Parts:
- removed the U1106 at (113.8, 90.6)
- added C1001: 100n, Capacitor_SMD:C_0603_1608Metric_Pad1.05x0.95mm_HandSolder, F.Cu at (50.4, 153.0)
- added C1006: 100n, Capacitor_SMD:C_0603_1608Metric_Pad1.05x0.95mm_HandSolder, F.Cu at (50.4, 155.5)
- added C1008: 1u, Capacitor_SMD:C_0603_1608Metric_Pad1.05x0.95mm_HandSolder, F.Cu at (49.0, 102.7)
- added C1101: 100n, Capacitor_SMD:C_0603_1608Metric_Pad1.05x0.95mm_HandSolder, F.Cu at (74.3, 100.7)
- added C1102: 10u, Capacitor_SMD:C_0805_2012Metric_Pad1.15x1.40mm_HandSolder, F.Cu at (74.5, 116.1)
- added C1104: 1u, Capacitor_SMD:C_0603_1608Metric_Pad1.05x0.95mm_HandSolder, F.Cu at (74.3, 118.8)
- added C1106: 100n, Capacitor_SMD:C_0603_1608Metric_Pad1.05x0.95mm_HandSolder, F.Cu at (74.3, 103.2)
- added C1114: 100n, Capacitor_SMD:C_0603_1608Metric_Pad1.05x0.95mm_HandSolder, F.Cu at (66.8, 111.3)
- added C705: 100n, Capacitor_SMD:C_0603_1608Metric_Pad1.05x0.95mm_HandSolder, F.Cu at (57.5, 71.2)
- added C706: 100n, Capacitor_SMD:C_0603_1608Metric_Pad1.05x0.95mm_HandSolder, F.Cu at (57.5, 73.8)
- added C819: 10p, Capacitor_SMD:C_0603_1608Metric_Pad1.05x0.95mm_HandSolder, F.Cu at (-2.29, 112.5)
- added C820: 10p, Capacitor_SMD:C_0603_1608Metric_Pad1.05x0.95mm_HandSolder, F.Cu at (-15.3, 112.3)
- added C821: 10p, Capacitor_SMD:C_0603_1608Metric_Pad1.05x0.95mm_HandSolder, F.Cu at (-2.09, 110.0)
- added C822: 10p, Capacitor_SMD:C_0603_1608Metric_Pad1.05x0.95mm_HandSolder, F.Cu at (-1.99, 107.5)
- added C908: 10p, Capacitor_SMD:C_0603_1608Metric_Pad1.05x0.95mm_HandSolder, F.Cu at (-30.8, 111.7)
- added C909: 10p, Capacitor_SMD:C_0603_1608Metric_Pad1.05x0.95mm_HandSolder, F.Cu at (-26.3, 105.0)
- added C910: 10p, Capacitor_SMD:C_0603_1608Metric_Pad1.05x0.95mm_HandSolder, F.Cu at (-30.7, 108.6)
- added M101: 60817-096, ETH1CLCR1:60817-096, F.Cu at (83.6, 134.5)
- added Q805: BC847W, Package_TO_SOT_SMD:SOT-323_SC-70, F.Cu at (-10.8, 109.2)
- added Q806: BC847W, Package_TO_SOT_SMD:SOT-323_SC-70, F.Cu at (-10.8, 105.6)
- added Q807: BC847W, Package_TO_SOT_SMD:SOT-323_SC-70, F.Cu at (-15.3, 109.2)
- added Q808: BC847W, Package_TO_SOT_SMD:SOT-323_SC-70, F.Cu at (-15.3, 105.6)
- added Q901: BC847W, Package_TO_SOT_SMD:SOT-323_SC-70, F.Cu at (-39.6, 112.3)
- added Q902: BC847W, Package_TO_SOT_SMD:SOT-323_SC-70, F.Cu at (-30.7, 105.6)
- added Q903: BC847W, Package_TO_SOT_SMD:SOT-323_SC-70, F.Cu at (-35.2, 112.3)
- added R844: 10k, Resistor_SMD:R_0603_1608Metric_Pad1.05x0.95mm_HandSolder, F.Cu at (-6.64, 112.3)
- added R845: 10k, Resistor_SMD:R_0603_1608Metric_Pad1.05x0.95mm_HandSolder, F.Cu at (-1.99, 105.0)
- added R846: 10k, Resistor_SMD:R_0603_1608Metric_Pad1.05x0.95mm_HandSolder, F.Cu at (-6.44, 108.6)
- added R847: 10k, Resistor_SMD:R_0603_1608Metric_Pad1.05x0.95mm_HandSolder, F.Cu at (-11.0, 112.3)
- added R948: 10k, Resistor_SMD:R_0603_1608Metric_Pad1.05x0.95mm_HandSolder, F.Cu at (-26.4, 108.6)
- added R949: 10k, Resistor_SMD:R_0603_1608Metric_Pad1.05x0.95mm_HandSolder, F.Cu at (-30.8, 114.3)
- added R950: 10k, Resistor_SMD:R_0603_1608Metric_Pad1.05x0.95mm_HandSolder, F.Cu at (-26.4, 111.2)
- added U1103: REF192, Package_SO:SSOP-8_3.9x5.05mm_P1.27mm, F.Cu at (67.9, 117.9)
- added U1107: AD8605, Package_TO_SOT_SMD:SOT-23-5_HandSoldering, F.Cu at (74.9, 107.8)
- added U917: ULN2003A, Package_SO:TSSOP-16_4.4x5mm_P0.65mm, F.Cu at (127.0, 65.7)
- C1510, C1512: value 2u2/50V -> 4u7/50V
- C713: renamed from C710; value 43p -> 43p/300V
- C810: value 1u -> 1u/150V; footprint Capacitor_SMD:C_0603_1608Metric_Pad1.05x0.95mm_HandSolder -> Capacitor_SMD:C_1812_4532Metric_Pad1.30x3.40mm_HandSolder
- C814: value 33p -> 33p/300V
- C815: value 6800p -> 6800p/200V
- Q701, Q702, Q703, Q704: value BC847W -> BC847; footprint Package_TO_SOT_SMD:SOT-323_SC-70 -> Package_TO_SOT_SMD:SOT-23; moved to F.Cu
- R1103, R1104: value 1k -> 10k
- R722: value 1k -> 2k2
- R820, R823: value 261 -> 261/.5W; footprint Resistor_SMD:R_0603_1608Metric_Pad1.05x0.95mm_HandSolder -> Resistor_SMD:R_0805_2012Metric_Pad1.15x1.40mm_HandSolder
- R821, R822: value 2R7 -> 2R7/.5W
- R824: value 90k/.01% -> RN732BTTD9002B25; footprint Resistor_SMD:R_0603_1608Metric_Pad1.05x0.95mm_HandSolder -> Resistor_SMD:R_1206_3216Metric_Pad1.42x1.75mm_HandSolder
- R825, R830: value 10k -> RN732ATTE1002B25
- R826: value 10 -> RP73PF2A10RBTDF; footprint Resistor_SMD:R_0603_1608Metric_Pad1.05x0.95mm_HandSolder -> Resistor_SMD:R_0805_2012Metric_Pad1.15x1.40mm_HandSolder
- R827: value 100 -> RT1206BRB07100RL; footprint Resistor_SMD:R_0603_1608Metric_Pad1.05x0.95mm_HandSolder -> Resistor_SMD:R_1206_3216Metric_Pad1.42x1.75mm_HandSolder
- R828: value 1k01 -> TNPW08051K01BEEA; footprint Resistor_SMD:R_0603_1608Metric_Pad1.05x0.95mm_HandSolder -> Resistor_SMD:R_0805_2012Metric_Pad1.15x1.40mm_HandSolder
- R829: value 1k111 -> RN73R2BTTD1001B25; footprint Resistor_SMD:R_0603_1608Metric_Pad1.05x0.95mm_HandSolder -> Resistor_SMD:R_1206_3216Metric_Pad1.42x1.75mm_HandSolder
- R831, R832, R833, R834, R835, R836, R837, R838, R925, R926, R927, R928, R929, R930, R936, R943, R945, R947: value 330 -> 680
- R906, R908, R909, R910, R911, R913, R917, R919: value 3k01/.1% -> RQ73C2A3K01BTDF; footprint Resistor_SMD:R_0603_1608Metric_Pad1.05x0.95mm_HandSolder -> Resistor_SMD:R_0805_2012Metric_Pad1.15x1.40mm_HandSolder
- R921, R923: value 900 -> PAT1206E9000BST1; footprint Resistor_SMD:R_0603_1608Metric_Pad1.05x0.95mm_HandSolder -> Resistor_SMD:R_1206_3216Metric_Pad1.42x1.75mm_HandSolder
- R922, R924: value 100 -> RN73R2BTTD1000B25; footprint Resistor_SMD:R_0603_1608Metric_Pad1.05x0.95mm_HandSolder -> Resistor_SMD:R_1206_3216Metric_Pad1.42x1.75mm_HandSolder
- U1004: value DAC7568ICPWR -> DAC8568IBPWR
- U1105: value AD8605 -> AD8606-2-MSOP; footprint Package_TO_SOT_SMD:SOT-23-5_HandSoldering -> Package_SO:MSOP-8_3x3mm_P0.65mm
- moved Q801 227.6 mm to (-6.39, 105.6), turned to 0 degrees
- moved Q702 132.3 mm to (53.3, 83.7), turned to 0 degrees
- moved Q701 132.0 mm to (53.3, 79.1), turned to 0 degrees
- moved Q703 127.5 mm to (57.8, 79.1), turned to 0 degrees
- moved Q704 123.4 mm to (62.2, 79.1), turned to 0 degrees
- moved U1105 44.2 mm to (68.3, 107.7), turned to 0 degrees
- moved C814 31.5 mm to (163.1, 34.5)
- moved R819 31.5 mm to (165.4, 34.5)
- moved L1502 20.1 mm to (111.9, 132.0), turned to 180 degrees
- moved U1502 15.0 mm to (111.6, 124.1), turned to 0 degrees
- moved R1409 14.4 mm to (89.5, 86.5)
- moved U1504 12.6 mm to (97.7, 107.3), turned to 180 degrees
- moved U1503 10.3 mm to (97.8, 123.8), turned to 180 degrees
- moved U1506 2.54 mm to (87.9, 68.3)
- moved C810 2.30 mm to (176.4, 63.4), turned to 0 degrees
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- renumbered C1001 to C1002, C1002 to C1003, C1003 to C1005, C1005 to C1007, C1006 to C1009, C1007 to C1010, C1008 to C1011, C1009 to C1012, C1010 to C1013, C1011 to C1014, C1012 to C1015, C1013 to C1016, C1014 to C1017, C1015 to C1018, C1016 to C1019, C1017 to C1020, C1018 to C1021, C1019 to C1022, C1020 to C1023, C1021 to C1024, C1101 to C1103, C1102 to C1105, C1104 to C1107, C1103 to C1108, C1105 to C1109, C1106 to C1110, C1108 to C1111, C1109 to C1112, C1107 to C1113, C1110 to C1115, C1111 to C1116, C1112 to C1117, C1115 to C1118, C1116 to C1119, C1113 to C1120, C1114 to C1121, C1117 to C1122, C1118 to C1123, C1119 to C1124, C1120 to C1125, C1121 to C1126, C1122 to C1127, C1123 to C1128, C1124 to C1129, C1125 to C1130, C712 to C707, C705 to C708, C706 to C709, C707 to C710, C708 to C711, C709 to C712, C711 to C714, R706 to R704, R707 to R705, R704 to R706, R705 to R707, U1103 to U1104, U1104 to U1106, U1107 to U1108, U1108 to U1109, U1109 to U1110, U1110 to U1111, U1111 to U1112, U1112 to U1113
Connections:
- net /FGEN Buffer/FB_CAP renamed /FGEN Buffer + Source resistor/FB_CAP
- net /FGEN Buffer/FB_CLK renamed /FGEN Buffer + Source resistor/FB_CLK
- net /FGEN Buffer/FB_RDY renamed /FGEN Buffer + Source resistor/FB_RDY
- net /FGEN Buffer/FB_SDI renamed /FGEN Buffer + Source resistor/FB_SDI
- net /FGEN Buffer/FB_SDO renamed /FGEN Buffer + Source resistor/FB_SDO
- net /FGEN Buffer/FB_~CS renamed /FGEN Buffer + Source resistor/FB_~CS
- net /FGEN Buffer/FB_~RST renamed /FGEN Buffer + Source resistor/FB_~RST
- net /FGEN Buffer/FGEN renamed /FGEN Buffer + Source resistor/FGEN
- net /FGEN Buffer/SR100CTR renamed /FGEN Buffer + Source resistor/SR100CTR
- net /FGEN Buffer/SR10CTR renamed /FGEN Buffer + Source resistor/SR10CTR
- net /FGEN Buffer/SR10KCTR renamed /FGEN Buffer + Source resistor/SR10KCTR
- net /FGEN Buffer/SR1KCTR renamed /FGEN Buffer + Source resistor/SR1KCTR
- net /FGEN Buffer/TRIM_3 renamed /FGEN Buffer + Source resistor/TRIM_3
- net /FGEN Buffer/VLI renamed /FGEN Buffer + Source resistor/VLI
- R831 pad 2: /MCU2/R10CRT -> +5VF
- R832 pad 2: /MCU2/R10CRT -> +5VF
- R833 pad 2: /MCU2/R100CRT -> +5VF
- R834 pad 2: /MCU2/R100CRT -> +5VF
- R835 pad 2: /MCU2/R1KCRT -> +5VF
- R836 pad 2: /MCU2/R1KCRT -> +5VF
- R837 pad 2: /MCU2/R10KCRT -> +5VF
- R838 pad 2: /MCU2/R10KCRT -> +5VF
- R925 pad 2: /MCU2/PA_MOS1 -> +5VF
- R926 pad 2: /MCU2/PA_MOS2 -> +5VF
- R927 pad 2: /MCU2/PA_MOS3 -> +5VF
- R928 pad 2: /MCU2/PA_MOS4 -> +5VF
- R929 pad 2: /MCU2/PA_MOS5 -> +5VF
- R930 pad 2: /MCU2/PA_MOS6 -> +5VF
- R936 pad 1: /MCU2/PA_50MV -> +5VF
- R943 pad 1: /MCU2/PA_50MV -> +5VF
- R945 pad 1: /MCU2/PA_EM -> +5VF
- R947 pad 1: /MCU2/PA_NULL -> +5VF
- U1105 pad 2: AGNDF -> /ADC/ADC_REF
- U1105 pad 4: /ADC/ADC_REF -> AGNDF
- U1105 pad 5: +5VF -> Net-(R1103-Pad1)
- U805 pad 2: AGNDF -> /Range Resistors/R10NPN
- U806 pad 2: AGNDF -> /Range Resistors/R10NPN
- U807 pad 2: AGNDF -> /Range Resistors/R100NPN
- U808 pad 2: AGNDF -> /Range Resistors/R100NPN
- U809 pad 2: AGNDF -> /Range Resistors/R1KNPN
- U810 pad 2: AGNDF -> /Range Resistors/R1KNPN
- U811 pad 2: AGNDF -> /Range Resistors/R10KNPN
- U812 pad 2: AGNDF -> /Range Resistors/R10KNPN
- U907 pad 2: AGNDF -> /Process Amplifier/MOS1
- U908 pad 2: AGNDF -> /Process Amplifier/MOS2
- U909 pad 2: AGNDF -> /Process Amplifier/MOS3
- U910 pad 2: AGNDF -> /Process Amplifier/MOS4
- U911 pad 2: AGNDF -> /Process Amplifier/MOS5
- U912 pad 2: AGNDF -> /Process Amplifier/MOS6
- U913 pad 2: AGNDF -> /Process Amplifier/50MV_NPN
- U914 pad 2: AGNDF -> /Process Amplifier/50MV_NPN
- U915 pad 2: AGNDF -> /Process Amplifier/EM_NPN
- U916 pad 2: AGNDF -> /Process Amplifier/NULL_NPN
