File: hardware/project/ETH1CLCR1/ETH1CLCR1.kicad_pcb (KiCad board)
At the start: 8 copper layers, 160 x 100 mm, 741 parts, among them J1201 C64AC, J1301 20021111-00010T4LF, J301 Conn_02x01, J302 20021111-00010T4LF, J601 20021111-00010T4LF, K1201 HE3621A0510, K1202 HE3621A0510, K1203 HE3621A0510, K1204 HE3621A0510, K1205 HE3621A0510, K1206 HE3621A0510, K701 9012, K702 9012, K703 9012, K704 9012, K801 TQ2SA-5V, Q1101 BC847W, Q1102 BC847W, Q1103 BC847W, Q1104 BC847W, Q501 IRFR5410, Q701 BC847W, Q702 BC847W, Q703 BC847W, Q704 BC847W, Q705 MMBT4401L, Q706 MMBT4403L, Q801 BC847W, Q802 2N2218A, Q803 2N2904A, Q804 BC847W, Q805 BC847W, Q806 BC847W, Q807 BC847W, Q808 BC847W, Q901 BC847W, Q902 BC847W, Q903 BC847W, U1001 TL074, U1002 TL074, U1003 REF192, U1004 DAC8568IBPWR, U1101 ADG419BR, U1102 ADG419BR, U1103 ADR4525BRZ, U1104 ADA4807-1AKSZ-R2, U1105 ADA4807-2ARM, U1106 AD7380, U1107 ADA4807-2ARM, U1108 LT6350, U1109 LT6350, U1110 OPA602, U1111 OPA602, U1112 PGA103, U1113 PGA103, U1201 ULN2003A, U1301 24LC08B-E/MS, U1302 STM32H743ZI, U1401 ECS-3225SMV-500-GP-TR, U1402 REF192, U1403 74AHCT1G08, U1404 AD5689BRUZ, U1405 AD9835, U1406 TL072, U1407 DG419LDY, U1408 AD5453YRMZ, U1409 LT1468, U1410 LT1468, U1411 LT1468, U1501 TSR2-2450, U1502 LM1117DTX-3.3/NOPB, U1503 LM1117DTX-3.3/NOPB, U1504 LT8330_S6, U1505 LT8330_S6, U1506 MC7815BD2TG, U1507 MC7915BD2TG, U1508 TSR1-2490, U1509 LM1117DTX-5.0/NOPB, U1510 MC78M12ABDTRKG, U1511 MC79M12CDTG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

Commit message: PCB layout
Parts:
- added C1139: 100n, Capacitor_SMD:C_0603_1608Metric_Pad1.05x0.95mm_HandSolder, B.Cu at (113.7, 87.1)
- added C1140: 100n, Capacitor_SMD:C_0603_1608Metric_Pad1.05x0.95mm_HandSolder, B.Cu at (89.9, 87.1)
- added C1201: 100n, Capacitor_SMD:C_0603_1608Metric_Pad1.05x0.95mm_HandSolder, B.Cu at (224.4, 78.1)
- moved C1103 6.06 mm to (108.1, 94.1), turned to 270 degrees
- moved R941 4.32 mm to (117.0, 64.8), turned to 90 degrees
- moved R1506 3.81 mm to (104.1, 134.7)
- moved C1420 2.54 mm to (128.5, 85.6)
- moved R1113 1.40 mm to (116.0, 87.1)
- moved C401 1.27 mm to (195.1, 91.7)
- moved D1502 1.27 mm to (104.6, 120.5)
- moved C1114 1.14 mm to (117.5, 87.1)
- moved C1514 1.14 mm to (104.8, 127.3)
- moved C1130 1.02 mm to (115.1, 69.3)
- moved C1519 0.76 mm to (104.6, 114.8)
- moved C1522 0.76 mm to (101.6, 114.8)
- moved D1501 0.68 mm to (95.4, 131.3)
- moved C1513 0.64 mm to (82.9, 132.6), turned to 180 degrees
- moved R1503 0.64 mm to (82.9, 132.6)
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Routing:
- net AGNDF: track 27.7 -> 78.8 mm, vias 19 -> 46
- net +5VF: track 27.7 -> 68.1 mm, vias 17 -> 32
- net -15VF: track 37.4 -> 73.3 mm, vias 23 -> 40
- net +15VF: track 29.2 -> 64.4 mm, vias 19 -> 37
- net Net-(U1110-Pad2): track 0.00 -> 30.4 mm
- net Net-(C1516-Pad1): track 0.00 -> 30.3 mm, vias 0 -> 8
- net +3.3VF: track 23.4 -> 50.1 mm, vias 15 -> 27
- net -12VF: track 13.2 -> 36.0 mm, vias 9 -> 20
- net +24VDD: track 72.8 -> 95.5 mm, vias 32 -> 47
- net Net-(D401-Pad3): track 0.00 -> 21.7 mm
- net +12VF: track 16.2 -> 37.1 mm, vias 11 -> 22
- net /Trigger/TRIG_OUT_SIGN: track 0.00 -> 17.4 mm, vias 0 -> 4
- net Net-(U1111-Pad2): track 0.00 -> 16.8 mm
- net /Trigger/TRIG_OUT_EN: track 0.00 -> 16.5 mm, vias 0 -> 2
- net Net-(U904-Pad3): track 0.00 -> 15.9 mm
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- added copper zone on B.Cu, net Net-(C1514-Pad1)
- added copper zone on F.Cu, net Net-(C1514-Pad1)
- added copper zone on B.Cu, net Net-(C1514-Pad2)
- added copper zone on F.Cu, net Net-(C1514-Pad2)
- added copper zone on B.Cu, net Net-(C1515-Pad1)
- added copper zone on F.Cu, net Net-(C1515-Pad1)
- added copper zone on B.Cu, net Net-(C1515-Pad2)
- added copper zone on F.Cu, net Net-(C1515-Pad2)
- added copper zone on Power_C, net Net-(C1516-Pad1)
- added copper zone on Power_B, net Net-(C1517-Pad1)
- removed copper zone on F.Cu, net (none)

Commit message: PCB layout
Parts:
- moved R1142 3.81 mm to (104.6, 83.9)
- moved C1138 3.81 mm to (104.6, 81.7)
- moved Q1104 3.81 mm to (104.6, 82.4)
- moved C1137 3.56 mm to (101.1, 81.5)
- moved Q1103 3.56 mm to (101.1, 82.3)
- moved R1141 3.56 mm to (101.1, 83.8)
- moved R1420 2.54 mm to (130.2, 75.2)
- moved R843 2.54 mm to (210.1, 78.5)
- moved R842 2.16 mm to (210.1, 76.2)
- moved R807 0.89 mm to (193.7, 56.9)
- moved R808 0.89 mm to (164.8, 50.7)
- moved R933 0.64 mm to (102.6, 58.2), turned to 0 degrees
- moved C824 0.51 mm to (195.5, 51.3)
- moved C805 0.38 mm to (174.6, 55.9)
- moved R812 0.38 mm to (195.5, 54.0)
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Connections:
- U1201 pad 1: /Connector/CXN_REL1 -> /Connector/CXN_REL6
- U1201 pad 11: Net-(K1206-Pad3) -> Net-(K1201-Pad3)
- U1201 pad 12: Net-(K1205-Pad3) -> Net-(K1202-Pad3)
- U1201 pad 13: Net-(K1204-Pad3) -> Net-(K1203-Pad3)
- U1201 pad 14: Net-(K1203-Pad3) -> Net-(K1204-Pad3)
- U1201 pad 15: Net-(K1202-Pad3) -> Net-(K1205-Pad3)
- U1201 pad 16: Net-(K1201-Pad3) -> Net-(K1206-Pad3)
- U1201 pad 2: /Connector/CXN_REL2 -> /Connector/CXN_REL5
- U1201 pad 3: /Connector/CXN_REL3 -> /Connector/CXN_REL4
- U1201 pad 4: /Connector/CXN_REL4 -> /Connector/CXN_REL3
- U1201 pad 5: /Connector/CXN_REL5 -> /Connector/CXN_REL2
- U1201 pad 6: /Connector/CXN_REL6 -> /Connector/CXN_REL1
Routing:
- net /Connector/HCUR: track 0.00 -> 104.7 mm, vias 0 -> 2
- net /Connector/LCUR: track 0.00 -> 92.1 mm
- net Net-(C708-Pad2): track 0.00 -> 53.6 mm, vias 0 -> 1
- net Net-(K801-Pad3): track 0.00 -> 43.9 mm
- net /FGEN Buffer + Source resistor/VLI: track 0.00 -> 36.2 mm, vias 0 -> 1
- net /Connector/HPOT: track 0.00 -> 35.1 mm
- net Net-(C708-Pad1): track 0.00 -> 32.0 mm, vias 0 -> 1
- net Net-(R906-Pad1): track 0.00 -> 29.1 mm, vias 0 -> 2
- net Net-(C811-Pad2): track 0.00 -> 28.3 mm, vias 0 -> 1
- net Net-(D805-Pad1): track 0.00 -> 25.8 mm
- net Net-(C907-Pad2): track 0.00 -> 23.9 mm, vias 0 -> 2
- net Net-(R921-Pad2): track 0.00 -> 22.9 mm, vias 0 -> 1
- net Net-(R808-Pad2): track 0.00 -> 22.8 mm, vias 0 -> 2
- net Net-(R908-Pad1): track 0.00 -> 21.1 mm, vias 0 -> 3
- net /Process Amplifier/Err: track 0.00 -> 18.7 mm
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- added copper zone on B.Cu, net Net-(D811-Pad1)
