File: hardware/project/ETH1CLCR1/Ethernet.sch (KiCad schematic (older format))
At the start: 43 parts, among them U201 LC03-3.3, U202 LAN8742A, U203 LC03-3.3, Y201 NX5032GA-25.000M-LN-CD-1

Commit message: Footprint asigment (not finished).
Parts:
- C203, C209: footprint Capacitor_SMD:C_0603_1608Metric_Pad1.05x0.95mm_HandSolder -> Capacitor_SMD:C_0805_2012Metric_Pad1.15x1.40mm_HandSolder
Changed lines of the file:
@@
 F 0 "C209" H 2765 1996 50  0000 L CNN
 F 1 "1u" H 2765 1905 50  0000 L CNN
-F 2 "Capacitor_SMD:C_0603_1608Metric_Pad1.05x0.95mm_HandSolder" H 2688 1800 50  0001 C CNN
+F 2 "Capacitor_SMD:C_0805_2012Metric_Pad1.15x1.40mm_HandSolder" H 2688 1800 50  0001 C CNN
 F 3 "~" H 2650 1950 50  0001 C CNN
 	1    2650 1950
@@
 F 0 "C203" H 3865 1296 50  0000 L CNN
 F 1 "1u" H 3865 1205 50  0000 L CNN
-F 2 "Capacitor_SMD:C_0603_1608Metric_Pad1.05x0.95mm_HandSolder" H 3788 1100 50  0001 C CNN
+F 2 "Capacitor_SMD:C_0805_2012Metric_Pad1.15x1.40mm_HandSolder" H 3788 1100 50  0001 C CNN
 F 3 "~" H 3750 1250 50  0001 C CNN
 	1    3750 1250

Commit message: Modification in schematic and PCB layout.
Parts:
- C203, C209: footprint Capacitor_SMD:C_0805_2012Metric_Pad1.15x1.40mm_HandSolder -> Capacitor_SMD:C_0603_1608Metric_Pad1.05x0.95mm_HandSolder
Changed lines of the file:
@@
 F 0 "C209" H 2765 1996 50  0000 L CNN
 F 1 "1u" H 2765 1905 50  0000 L CNN
-F 2 "Capacitor_SMD:C_0805_2012Metric_Pad1.15x1.40mm_HandSolder" H 2688 1800 50  0001 C CNN
+F 2 "Capacitor_SMD:C_0603_1608Metric_Pad1.05x0.95mm_HandSolder" H 2688 1800 50  0001 C CNN
 F 3 "~" H 2650 1950 50  0001 C CNN
 	1    2650 1950
@@
 F 0 "C203" H 3865 1296 50  0000 L CNN
 F 1 "1u" H 3865 1205 50  0000 L CNN
-F 2 "Capacitor_SMD:C_0805_2012Metric_Pad1.15x1.40mm_HandSolder" H 3788 1100 50  0001 C CNN
+F 2 "Capacitor_SMD:C_0603_1608Metric_Pad1.05x0.95mm_HandSolder" H 3788 1100 50  0001 C CNN
 F 3 "~" H 3750 1250 50  0001 C CNN
 	1    3750 1250

Commit message: Redesinged ADC schematic.
Parts:
- renumbered C213 to C201, C201 to C202, C208 to C203, C214 to C204, C202 to C205, C209 to C206, C203 to C207, C204 to C208, C205 to C209, C206 to C210, C207 to C211, C210 to C212, C212 to C213, C211 to C214, R205 to R201, R206 to R202, R207 to R203, R208 to R204, R212 to R205, R217 to R206, R218 to R207, R219 to R208, R220 to R209, R221 to R210, R213 to R211, R209 to R212, R214 to R213, R215 to R214, R201 to R215, R202 to R216, R203 to R217, R204 to R218, R216 to R219, R210 to R220, R211 to R221, U202 to U201, U201 to U202
