File: hardware/project/ETH1CLCR1/ProcessAmplifier.sch (KiCad schematic (older format))
At the start: 32 parts, among them U1401 RC4558, U1402 RC4558, U1403 LF356, U1404 LF356

Commit message: Schematic design
Parts:
- added C1406, C?: C, symbol Device:C
- added D1403, D1404: D_Zener, symbol Device:D_Zener
- added R1420, R1421, R1424, R1425, R1426, R1427, R1428, R1429, R1431, R1433, R1435, R1436, R1437, R1438, R1439, R1440, R1441, R? (x6): R, symbol Device:R
- added R1430: 1k, symbol Device:R
- added R1432: 1M, symbol Device:R
- added R1434: 10k, symbol Device:R
- added U1405, U1406, U1407, U1408, U1409, U1410, U1413, U? (x3): TLP3542, Package_DIP:DIP-5-6_W7.62mm, symbol Relay_SolidState:TLP3542
- added U1411, U1412: RC4558, symbol Amplifier_Operational:RC4558
- added U? (x2): AD5290YRMZ10, Package_SO:MSOP-10_3x3mm_P0.5mm, symbol Potentiometer_Digital:AD5290
- added U? (x2): AD5293BRUZ-100, Package_SO:TSSOP-14_4.4x5mm_P0.65mm, symbol Potentiometer_Digital:AD5293
- gave numbers to parts that had none: 2
Connections:
- net labels added: +12VF, +3.3VP, -12VF, Em, OFS3, OFS4, OSF1, OSF2, OSF3, OSF4
- wire segments 87 -> 212
Other:
- moved on the sheet: C1401, C1402, C1403, C1404, C1405, D1401, D1402, R1401, R1402, R1403, R1404, R1405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

Commit message: Schematic design
Parts:
- removed D1401, D1402: 1N4148, symbol Device:D
- removed U1405, U1406, U1407, U1408, U1409, U1410, U1413, U? (x3): TLP3542, Package_DIP:DIP-5-6_W7.62mm, symbol Relay_SolidState:TLP3542
- removed U? (x2): AD5290YRMZ10, Package_SO:MSOP-10_3x3mm_P0.5mm, symbol Potentiometer_Digital:AD5290
- removed U? (x2): AD5293BRUZ-100, Package_SO:TSSOP-14_4.4x5mm_P0.65mm, symbol Potentiometer_Digital:AD5293
- added D1401: BAT54SW, Package_TO_SOT_SMD:SOT-323_SC-70, symbol Diode:BAT54SW
- added RV1401, RV1402: 10k, Resistor_SMD:R_0603_1608Metric_Pad1.05x0.95mm_HandSolder, symbol Device:R_POT_TRIM
- added RV1403, RV1404: 100k, Resistor_SMD:R_0603_1608Metric_Pad1.05x0.95mm_HandSolder, symbol Device:R_POT_TRIM
- added U1405, U1406, U1407, U1408, U1409, U1410, U1413, U1414, U1415, U1416: AQY212GS, symbol ETH1CLCR1:AQY212GS
- C1401: value C -> 100n; footprint (none) -> Capacitor_SMD:C_0603_1608Metric_Pad1.05x0.95mm_HandSolder
- C1403: value C -> 7p5; footprint (none) -> Capacitor_SMD:C_0603_1608Metric_Pad1.05x0.95mm_HandSolder
- C1406: value C -> 220p
- R1401, R1419: value R -> 1M; footprint (none) -> Resistor_SMD:R_0603_1608Metric_Pad1.05x0.95mm_HandSolder
- R1403, R1406, R1440: value R -> 10k; footprint (none) -> Resistor_SMD:R_0603_1608Metric_Pad1.05x0.95mm_HandSolder
- R1407, R1408, R1409, R1410, R1412, R1415, R1438: value R -> 3k01/.05%
- R1411, R1413, R1414, R1417: value R -> NC; footprint (none) -> Resistor_SMD:R_0603_1608Metric_Pad1.05x0.95mm_HandSolder
- R1416: value R -> 1M
- R1418: value 5k01 -> 3k01/.05%
- R1420, R1422: value R -> 900; footprint (none) -> Resistor_SMD:R_0603_1608Metric_Pad1.05x0.95mm_HandSolder
- R1421, R1423: value R -> 100; footprint (none) -> Resistor_SMD:R_0603_1608Metric_Pad1.05x0.95mm_HandSolder
- R1424, R1425, R1426, R1427, R1428, R1429, R1435: value R -> 330; footprint (none) -> Resistor_SMD:R_0603_1608Metric_Pad1.05x0.95mm_HandSolder
- R1430, R1432, R1434: footprint (none) -> Resistor_SMD:R_0603_1608Metric_Pad1.05x0.95mm_HandSolder
- R1431, R1436, R1439, R1441: value R -> 1k; footprint (none) -> Resistor_SMD:R_0603_1608Metric_Pad1.05x0.95mm_HandSolder
- R1433: value R -> 22k; footprint (none) -> Resistor_SMD:R_0603_1608Metric_Pad1.05x0.95mm_HandSolder
- R1437: value R -> 100k; footprint (none) -> Resistor_SMD:R_0603_1608Metric_Pad1.05x0.95mm_HandSolder
- R1442: renamed from R?; value R -> 10k; footprint (none) -> Resistor_SMD:R_0603_1608Metric_Pad1.05x0.95mm_HandSolder
- R1443: renamed from R?; value R -> 1k; footprint (none) -> Resistor_SMD:R_0603_1608Metric_Pad1.05x0.95mm_HandSolder
- R1444: renamed from R?; value R -> 22k; footprint (none) -> Resistor_SMD:R_0603_1608Metric_Pad1.05x0.95mm_HandSolder
- R1445, R1446, R1447: renamed from R?; value R -> 330; footprint (none) -> Resistor_SMD:R_0603_1608Metric_Pad1.05x0.95mm_HandSolder
- gave numbers to parts that had none: 1
Connections:
- net labels added: Eref, HPOT, LCUR, LPOT, PA_50MV, PA_EM, PA_MOS1, PA_MOS2, PA_MOS3, PA_MOS4, PA_MOS5, PA_MOS6, PA_NULL, PA_OFS1, PA_OFS2, PA_OFS3, PA_OFS4
- net labels removed: +15VF, +3.3VP, -15VF, Hp, Lc, Lp, OFS3, OFS4, OSF1, OSF2, OSF3, OSF4
- wire segments 212 -> 213
Other:
- moved on the sheet: C1401, C1402, C1403, C1404, C1405, C1406, C1407, D1403, D1404, R1401, R1402, R1403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

Commit message: Need to redesign the AC source, the LT1468 is too slow.
Parts:
- C1402: value C -> 100n
- C1404: value CTRIM -> 2-8p
- C1405: value C -> 15p
- C1407: value C -> 390p
- R1402: value R -> 1M
- R1404, R1405: value R -> 10k
Changed lines of the file:
@@
 P 2200 5100
 F 0 "C1402" V 1948 5100 50  0000 C CNN
-F 1 "C" V 2039 5100 50  0000 C CNN
+F 1 "100n" V 2039 5100 50  0000 C CNN
 F 2 "" H 2238 4950 50  0001 C CNN
 F 3 "~" H 2200 5100 50  0001 C CNN
@@
 P 2450 5350
 F 0 "R1402" H 2520 5396 50  0000 L CNN
-F 1 "R" H 2520 5305 50  0000 L CNN
+F 1 "1M" H 2520 5305 50  0000 L CNN
 F 2 "" V 2380 5350 50  0001 C CNN
 F 3 "~" H 2450 5350 50  0001 C CNN
@@
 P 2700 5100
 F 0 "R1405" V 2493 5100 50  0000 C CNN
-F 1 "R" V 2584 5100 50  0000 C CNN
+F 1 "10k" V 2584 5100 50  0000 C CNN
 F 2 "" V 2630 5100 50  0001 C CNN
 F 3 "~" H 2700 5100 50  0001 C CNN
@@
 P 2950 5350
 F 0 "C1404" H 3066 5396 50  0000 L CNN
-F 1 "CTRIM" H 3066 5305 50  0000 L CNN
+F 1 "2-8p" H 3066 5305 50  0000 L CNN
 F 2 "" H 2950 5350 50  0001 C CNN
 F 3 "~" H 2950 5350 50  0001 C CNN
@@
 P 2700 3500
 F 0 "R1404" V 2493 3500 50  0000 C CNN
-F 1 "R" V 2584 3500 50  0000 C CNN
+F 1 "10k" V 2584 3500 50  0000 C CNN
 F 2 "" V 2630 3500 50  0001 C CNN
 F 3 "~" H 2700 3500 50  0001 C CNN
@@
 P 3150 6850
 F 0 "C1405" H 3265 6896 50  0000 L CNN
-F 1 "C" H 3265 6805 50  0000 L CNN
+F 1 "15p" H 3265 6805 50  0000 L CNN
 F 2 "" H 3188 6700 50  0001 C CNN
 F 3 "~" H 3150 6850 50  0001 C CNN
@@
 P 10350 5600
 F 0 "C1407" H 10465 5646 50  0000 L CNN
-F 1 "C" H 10465 5555 50  0000 L CNN
+F 1 "390p" H 10465 5555 50  0000 L CNN
 F 2 "" H 10388 5450 50  0001 C CNN
 F 3 "~" H 10350 5600 50  0001 C CNN

Commit message: Footprint asigment (not finished).
Parts:
- removed U1403, U1404: LF356, symbol Amplifier_Operational:LF356
- added U1307, U1315: TL071, Package_SO:SOIC-8_3.9x4.9mm_P1.27mm, symbol Amplifier_Operational:TL071
- C1301: renamed from C1406; footprint (none) -> Capacitor_SMD:C_0603_1608Metric_Pad1.05x0.95mm_HandSolder
- C1302: renamed from C1402; footprint (none) -> Capacitor_SMD:C_0603_1608Metric_Pad1.05x0.95mm_HandSolder
- C1303: renamed from C1404; value 2-8p -> JZ100
- C1304: renamed from C1407; footprint (none) -> Capacitor_SMD:C_0603_1608Metric_Pad1.05x0.95mm_HandSolder
- C1305: renamed from C1405; footprint (none) -> Capacitor_SMD:C_0603_1608Metric_Pad1.05x0.95mm_HandSolder
- R1310: renamed from R1404; footprint (none) -> Resistor_SMD:R_0603_1608Metric_Pad1.05x0.95mm_HandSolder
- R1312: renamed from R1407; value 3k01/.05% -> 3k01/.1%; footprint (none) -> Resistor_SMD:R_0603_1608Metric_Pad1.05x0.95mm_HandSolder
- R1313: renamed from R1416; footprint (none) -> Resistor_SMD:R_0603_1608Metric_Pad1.05x0.95mm_HandSolder
- R1314: renamed from R1412; value 3k01/.05% -> 3k01/.1%; footprint (none) -> Resistor_SMD:R_0603_1608Metric_Pad1.05x0.95mm_HandSolder
- R1320: renamed from R1405; footprint (none) -> Resistor_SMD:R_0603_1608Metric_Pad1.05x0.95mm_HandSolder
- R1322: renamed from R1408; value 3k01/.05% -> 3k01/.1%; footprint (none) -> Resistor_SMD:R_0603_1608Metric_Pad1.05x0.95mm_HandSolder
- R1323: renamed from R1418; value 3k01/.05% -> 3k01/.1%; footprint (none) -> Resistor_SMD:R_0603_1608Metric_Pad1.05x0.95mm_HandSolder
- R1324: renamed from R1402; footprint (none) -> Resistor_SMD:R_0603_1608Metric_Pad1.05x0.95mm_HandSolder
- R1331: renamed from R1438; value 3k01/.05% -> 3k01/.1%; footprint (none) -> Resistor_SMD:R_0603_1608Metric_Pad1.05x0.95mm_HandSolder
- R1337: renamed from R1409; value 3k01/.05% -> 3k01/.1%; footprint (none) -> Resistor_SMD:R_0603_1608Metric_Pad1.05x0.95mm_HandSolder
- R1345: renamed from R1410; value 3k01/.05% -> 3k01/.1%; footprint (none) -> Resistor_SMD:R_0603_1608Metric_Pad1.05x0.95mm_HandSolder
- R1346: renamed from R1415; value 3k01/.05% -> 3k01/.1%; footprint (none) -> Resistor_SMD:R_0603_1608Metric_Pad1.05x0.95mm_HandSolder
- U1301: renamed from U1405; footprint (none) -> ETH1CLCR1:AQY212GS
- U1302: renamed from U1411; value RC4558 -> TL072; footprint (none) -> Package_SO:SOIC-8_3.9x4.9mm_P1.27mm; symbol Amplifier_Operational:RC4558 -> Amplifier_Operational:TL072
- U1303: renamed from U1406; footprint (none) -> ETH1CLCR1:AQY212GS
- U1304: renamed from U1401; value RC4558 -> TL072; footprint (none) -> Package_SO:SOIC-8_3.9x4.9mm_P1.27mm; symbol Amplifier_Operational:RC4558 -> Amplifier_Operational:TL072
- U1305: renamed from U1413; footprint (none) -> ETH1CLCR1:AQY212GS
- U1306: renamed from U1407; footprint (none) -> ETH1CLCR1:AQY212GS
- U1308: renamed from U1408; footprint (none) -> ETH1CLCR1:AQY212GS
- U1309: renamed from U1412; value RC4558 -> TL072; footprint (none) -> Package_SO:SOIC-8_3.9x4.9mm_P1.27mm; symbol Amplifier_Operational:RC4558 -> Amplifier_Operational:TL072
- U1310: renamed from U1415; footprint (none) -> ETH1CLCR1:AQY212GS
- U1311: renamed from U1416; footprint (none) -> ETH1CLCR1:AQY212GS
- U1312: renamed from U1402; value RC4558 -> TL072; footprint (none) -> Package_SO:SOIC-8_3.9x4.9mm_P1.27mm; symbol Amplifier_Operational:RC4558 -> Amplifier_Operational:TL072
- U1313: renamed from U1414; footprint (none) -> ETH1CLCR1:AQY212GS
- U1314: renamed from U1409; footprint (none) -> ETH1CLCR1:AQY212GS
- U1316: renamed from U1410; footprint (none) -> ETH1CLCR1:AQY212GS
- renumbered C1401 to C1306, C1403 to C1307, D1403 to D1301, D1404 to D1302, D1401 to D1303, R1440 to R1301, R1424 to R1302, R1436 to R1303, R1441 to R1304, R1411 to R1305, R1425 to R1306, R1433 to R1307, R1437 to R1308, R1439 to R1309, R1431 to R1311, R1435 to R1315, R1426 to R1316, R1420 to R1317, R1417 to R1318, R1421 to R1319, R1427 to R1321, R1442 to R1325, R1434 to R1326, R1447 to R1327, R1444 to R1328, R1430 to R1329, R1432 to R1330, R1443 to R1332, R1413 to R1333, R1446 to R1334, R1406 to R1335, R1445 to R1336, R1419 to R1338, R1428 to R1339, R1422 to R1340, R1414 to R1341, R1423 to R1342, R1403 to R1343, R1429 to R1344, R1401 to R1347, RV1404 to RV1301, RV1401 to RV1302, RV1403 to RV1303, RV1402 to RV1304
Connections:
- net +12VF: now also U1307.7 (V+), U1315.7 (V+)
- net -12VF: now also U1307.4 (V-), U1315.4 (V-)
- net at C1307.1, D1303.3, R1343.1: now also U1315.3 (+)
- net at C1303.1, R1320.1: now also U1307.3 (+)
- net at R1322.2: now also U1307.2 (-), U1307.6
- net at R1345.2: now also U1315.2 (-), U1315.6

Commit message: Modification in schematic and PCB layout.
Parts:
- C1303: footprint (none) -> ETH1CLCR1:JZ
- D1301, D1302: value D_Zener -> MM5Z5V1T5G; footprint (none) -> Diode_SMD:D_SOD-523
- RV1301, RV1303: value 100k -> 3314J-2-104E; footprint Resistor_SMD:R_0603_1608Metric_Pad1.05x0.95mm_HandSolder -> Potentiometer_SMD:Potentiometer_Bourns_3314J_Vertical
- RV1302, RV1304: value 10k -> 3314J-1-103E; footprint Resistor_SMD:R_0603_1608Metric_Pad1.05x0.95mm_HandSolder -> Potentiometer_SMD:Potentiometer_Bourns_3314J_Vertical
Other:
- moved on the sheet: D1301, D1302, R1307, RV1304
Changed lines of the file:
@@
 F 0 "C1303" H 3066 5396 50  0000 L CNN
 F 1 "JZ100" H 3066 5305 50  0000 L CNN
-F 2 "" H 2950 5350 50  0001 C CNN
+F 2 "ETH1CLCR1:JZ" H 2950 5350 50  0001 C CNN
 F 3 "~" H 2950 5350 50  0001 C CNN
 	1    2950 5350
@@
 Connection ~ 5550 7550
 Wire Wire Line
-	5550 7550 6400 7550
+	5550 7550 6450 7550
 Wire Wire Line
 	6600 7900 6600 7950
@@
 $EndComp
 Wire Wire Line
-	6600 4350 6050 4350
+	6600 4350 6200 4350
 Connection ~ 5550 4350
 Wire Wire Line
@@
 	7250 2500 7200 2500
 Wire Wire Line
-	6400 2850 8200 2850
-Connection ~ 6400 7550
-Wire Wire Line
-	6400 7550 6600 7550
-Wire Wire Line
-	6050 2200 6050 4350
-Wire Wire Line
-	6050 2200 8200 2200
-Connection ~ 6050 4350
-Wire Wire Line
-	6050 4350 5550 4350
+	6450 2850 8200 2850
+Connection ~ 6450 7550
+Wire Wire Line
+	6450 7550 6600 7550
+Wire Wire Line
+	6200 2200 6200 4350
+Wire Wire Line
+	6200 2200 8200 2200
+Connection ~ 6200 4350
+Wire Wire Line
+	6200 4350 5550 4350
 $Comp
 L Amplifier_Operational:TL072 U1302
@@
 L Device:R R1307
 U 1 1 5E114CA1
-P 9500 3300
-F 0 "R1307" V 9293 3300 50  0000 C CNN
-F 1 "22k" V 9384 3300 50  0000 C CNN
-F 2 "Resistor_SMD:R_0603_1608Metric_Pad1.05x0.95mm_HandSolder" V 9430 3300 50  0001 C CNN
-F 3 "~" H 9500 3300 50  0001 C CNN
-	1    9500 3300
+P 9500 3250
+F 0 "R1307" V 9293 3250 50  0000 C CNN
+F 1 "22k" V 9384 3250 50  0000 C CNN
+F 2 "Resistor_SMD:R_0603_1608Metric_Pad1.05x0.95mm_HandSolder" V 9430 3250 50  0001 C CNN
+F 3 "~" H 9500 3250 50  0001 C CNN
+	1    9500 3250
 	0    1    1    0
 $EndComp
@@
 $EndComp
 Wire Wire Line
-	9150 3400 9150 3300
+	9150 3400 9150 3250
 Wire Wire Line
 	9150 2900 9200 2900
 Wire Wire Line
-	9350 3300 9150 3300
-Connection ~ 9150 3300
-Wire Wire Line
-	9150 3300 9150 2900
-Wire Wire Line
-	9650 3300 9850 3300
-Wire Wire Line
-	9850 3300 9850 2800
+	9350 3250 9150 3250
+Connection ~ 9150 3250
+Wire Wire Line
+	9150 3250 9150 2900
+Wire Wire Line
+	9650 3250 9850 3250
+Wire Wire Line
+	9850 3250 9850 2800
 Wire Wire Line
 	9850 2800 9800 2800
@@
 L Device:D_Zener D1301
 U 1 1 5E17F019
-P 11550 1550
-F 0 "D1301" H 11550 1766 50  0000 C CNN
-F 1 "D_Zener" H 11550 1675 50  0000 C CNN
-F 2 "" H 11550 1550 50  0001 C CNN
-F 3 "~" H 11550 1550 50  0001 C CNN
-	1    11550 1550
+P 11500 1550
+F 0 "D1301" H 11500 1766 50  0000 C CNN
+F 1 "MM5Z5V1T5G" H 11500 1675 50  0000 C CNN
+F 2 "Diode_SMD:D_SOD-523" H 11500 1550 50  0001 C CNN
+F 3 "~" H 11500 1550 50  0001 C CNN
+	1    11500 1550
 	1    0    0    -1
 $EndComp
@@
 L Device:D_Zener D1302
 U 1 1 5E17F4C6
-P 11950 1550
-F 0 "D1302" H 11950 1766 50  0000 C CNN
-F 1 "D_Zener" H 11950 1675 50  0000 C CNN
-F 2 "" H 11950 1550 50  0001 C CNN
-F 3 "~" H 11950 1550 50  0001 C CNN
-	1    11950 1550
+P 12050 1550
+F 0 "D1302" H 12050 1766 50  0000 C CNN
+F 1 "MM5Z5V1T5G" H 12050 1675 50  0000 C CNN
+F 2 "Diode_SMD:D_SOD-523" H 12050 1550 50  0001 C CNN
+F 3 "~" H 12050 1550 50  0001 C CNN
+	1    12050 1550
 	-1   0    0    -1
 $EndComp
@@
 	11300 1900 11300 1550
 Wire Wire Line
-	11300 1550 11400 1550
+	11300 1550 11350 1550
 Wire Wire Line
 	12250 1550 12250 1900
 Wire Wire Line
-	11700 1550 11800 1550
-Wire Wire Line
-	12100 1550 12250 1550
+	11650 1550 11900 1550
+Wire Wire Line
+	12200 1550 12250 1550
 Connection ~ 11300 1900
 Connection ~ 12250 1900
@@
 	9350 5900 8900 5900
 Wire Wire Line
-	6400 7550 6400 2850
+	6450 7550 6450 2850
 Wire Wire Line
 	3600 6850 3600 7050
@@
 	10750 3300 10650 3300
 Wire Wire Line
-	5650 6750 5500 6750
+	5600 6750 5500 6750
 Wire Wire Line
 	5350 3600 5200 3600
@@
 P 5500 3600
 F 0 "RV1302" H 5430 3646 50  0000 R CNN
-F 1 "10k" H 5430 3555 50  0000 R CNN
-F 2 "Resistor_SMD:R_0603_1608Metric_Pad1.05x0.95mm_HandSolder" H 5500 3600 50  0001 C CNN
+F 1 "3314J-1-103E" H 5430 3555 50  0000 R CNN
+F 2 "Potentiometer_SMD:Potentiometer_Bourns_3314J_Vertical" H 5500 3600 50  0001 C CNN
 F 3 "~" H 5500 3600 50  0001 C CNN
 	1    5500 3600
@@
 L Device:R_POT_TRIM RV1304
 U 1 1 5E152712
-P 5800 6750
-F 0 "RV1304" H 5730 6796 50  0000 R CNN
-F 1 "10k" H 5730 6705 50  0000 R CNN
-F 2 "Resistor_SMD:R_0603_1608Metric_Pad1.05x0.95mm_HandSolder" H 5800 6750 50  0001 C CNN
-F 3 "~" H 5800 6750 50  0001 C CNN
-	1    5800 6750
+P 5750 6750
+F 0 "RV1304" H 5680 6796 50  0000 R CNN
+F 1 "3314J-1-103E" H 5680 6705 50  0000 R CNN
+F 2 "Potentiometer_SMD:Potentiometer_Bourns_3314J_Vertical" H 5750 6750 50  0001 C CNN
+F 3 "~" H 5750 6750 50  0001 C CNN
+	1    5750 6750
 	-1   0    0    -1
 $EndComp
@@
 L ETH1CLCR1:-12VF #PWR01325
 U 1 1 5E152718
-P 5800 6600
-F 0 "#PWR01325" H 5800 6450 50  0001 C CNN
-F 1 "-12VF" H 5815 6773 50  0000 C CNN
-F 2 "" H 5800 6600 50  0001 C CNN
-F 3 "" H 5800 6600 50  0001 C CNN
-	1    5800 6600
+P 5750 6600
+F 0 "#PWR01325" H 5750 6450 50  0001 C CNN
+F 1 "-12VF" H 5765 6773 50  0000 C CNN
+F 2 "" H 5750 6600 50  0001 C CNN
+F 3 "" H 5750 6600 50  0001 C CNN
+	1    5750 6600
 	1    0    0    -1
 $EndComp
@@
 L ETH1CLCR1:+12VF #PWR01329
 U 1 1 5E15271E
-P 5800 6900
-F 0 "#PWR01329" H 5800 6750 50  0001 C CNN
-F 1 "+12VF" H 5815 7073 50  0000 C CNN
-F 2 "" H 5800 6900 50  0001 C CNN
-F 3 "" H 5800 6900 50  0001 C CNN
-	1    5800 6900
+P 5750 6900
+F 0 "#PWR01329" H 5750 6750 50  0001 C CNN
+F 1 "+12VF" H 5765 7073 50  0000 C CNN
+F 2 "" H 5750 6900 50  0001 C CNN
+F 3 "" H 5750 6900 50  0001 C CNN
+	1    5750 6900
 	-1   0    0    1
 $EndComp
@@
 P 9350 6650
 F 0 "RV1303" V 9235 6650 50  0000 C CNN
-F 1 "100k" V 9144 6650 50  0000 C CNN
-F 2 "Resistor_SMD:R_0603_1608Metric_Pad1.05x0.95mm_HandSolder" H 9350 6650 50  0001 C CNN
+F 1 "3314J-2-104E" V 9144 6650 50  0000 C CNN
+F 2 "Potentiometer_SMD:Potentiometer_Bourns_3314J_Vertical" H 9350 6650 50  0001 C CNN
 F 3 "~" H 9350 6650 50  0001 C CNN
 	1    9350 6650
@@
 P 10400 3300
 F 0 "RV1301" H 10331 3346 50  0000 R CNN
-F 1 "100k" H 10331 3255 50  0000 R CNN
-F 2 "Resistor_SMD:R_0603_1608Metric_Pad1.05x0.95mm_HandSolder" H 10400 3300 50  0001 C CNN
+F 1 "3314J-2-104E" H 10331 3255 50  0000 R CNN
+F 2 "Potentiometer_SMD:Potentiometer_Bourns_3314J_Vertical" H 10400 3300 50  0001 C CNN
 F 3 "~" H 10400 3300 50  0001 C CNN
 	1    10400 3300

Commit message: Redesinged ADC schematic.
Parts:
- renumbered C1306 to C1301, C1307 to C1303, C1303 to C1304, C1304 to C1306, C1301 to C1307, D1303 to D1301, D1301 to D1302, D1302 to D1303, R1347 to R1301, R1324 to R1302, R1343 to R1303, R1310 to R1304, R1320 to R1305, R1331 to R1306, R1335 to R1307, R1312 to R1308, R1322 to R1309, R1337 to R1310, R1345 to R1311, R1305 to R1312, R1314 to R1313, R1313 to R1314, R1333 to R1315, R1318 to R1316, R1323 to R1317, R1341 to R1318, R1346 to R1319, R1338 to R1320, R1317 to R1321, R1319 to R1322, R1340 to R1323, R1342 to R1324, R1302 to R1325, R1306 to R1326, R1316 to R1327, R1321 to R1328, R1339 to R1329, R1344 to R1330, R1329 to R1331, R1311 to R1332, R1330 to R1333, R1307 to R1334, R1326 to R1335, R1315 to R1336, R1303 to R1337, R1325 to R1338, R1308 to R1339, R1332 to R1340, R1328 to R1341, R1309 to R1342, R1336 to R1343, R1301 to R1344, R1334 to R1345, R1304 to R1346, R1327 to R1347, RV1302 to RV1301, RV1304 to RV1302, RV1301 to RV1304, U1304 to U1301, U1312 to U1302, U1302 to U1303, U1309 to U1304, U1307 to U1305, U1315 to U1306, U1301 to U1307, U1303 to U1308, U1306 to U1309, U1308 to U1310, U1314 to U1311, U1316 to U1312, U1305 to U1313, U1313 to U1314, U1310 to U1315, U1311 to U1316

Commit message: Redesigned the power supply, added humidy+temp. sensor.
Parts:
- renumbered C1301 to C901, C1302 to C902, C1303 to C903, C1304 to C904, C1305 to C905, C1306 to C906, C1307 to C907, D1301 to D901, D1302 to D902, D1303 to D903, R1301 to R901, R1302 to R902, R1303 to R903, R1304 to R904, R1305 to R905, R1306 to R906, R1307 to R907, R1308 to R908, R1309 to R909, R1310 to R910, R1311 to R911, R1312 to R912, R1313 to R913, R1314 to R914, R1315 to R915, R1316 to R916, R1317 to R917, R1318 to R918, R1319 to R919, R1320 to R920, R1321 to R921, R1322 to R922, R1323 to R923, R1324 to R924, R1325 to R925, R1326 to R926, R1327 to R927, R1328 to R928, R1329 to R929, R1330 to R930, R1331 to R931, R1332 to R932, R1333 to R933, R1334 to R934, R1335 to R935, R1336 to R936, R1337 to R937, R1338 to R938, R1339 to R939, R1340 to R940, R1341 to R941, R1342 to R942, R1343 to R943, R1344 to R944, R1345 to R945, R1346 to R946, R1347 to R947, RV1301 to RV901, RV1302 to RV902, RV1303 to RV903, RV1304 to RV904, U1301 to U901, U1302 to U902, U1303 to U903, U1304 to U904, U1305 to U905, U1306 to U906, U1307 to U907, U1308 to U908, U1309 to U909, U1310 to U910, U1311 to U911, U1312 to U912, U1313 to U913, U1314 to U914, U1315 to U915, U1316 to U916

Commit message: Changes in schematics.
Parts:
- added C908, C909, C910: 10p, Capacitor_SMD:C_0603_1608Metric_Pad1.05x0.95mm_HandSolder, symbol Device:C
- added Q901, Q902, Q903: BC847W, Package_TO_SOT_SMD:SOT-323_SC-70, symbol Transistor_BJT:BC847W
- added R948, R949, R950: 10k, Resistor_SMD:R_0603_1608Metric_Pad1.05x0.95mm_HandSolder, symbol Device:R
- added U917: ULN2003A, Package_SO:TSSOP-16_4.4x5mm_P0.65mm, symbol Transistor_Array:ULN2003A
- R906, R908, R909, R910, R911, R913, R917, R919: value 3k01/.1% -> RQ73C2A3K01BTDF; footprint Resistor_SMD:R_0603_1608Metric_Pad1.05x0.95mm_HandSolder -> Resistor_SMD:R_0805_2012Metric_Pad1.15x1.40mm_HandSolder
- R921, R923: value 900 -> PAT1206E9000BST1; footprint Resistor_SMD:R_0603_1608Metric_Pad1.05x0.95mm_HandSolder -> Resistor_SMD:R_1206_3216Metric_Pad1.42x1.75mm_HandSolder
- R922, R924: value 100 -> RN73R2BTTD1000B25; footprint Resistor_SMD:R_0603_1608Metric_Pad1.05x0.95mm_HandSolder -> Resistor_SMD:R_1206_3216Metric_Pad1.42x1.75mm_HandSolder
- R925, R926, R927, R928, R929, R930, R936, R943, R945, R947: value 330 -> 680
Connections:
- net AGNDF: now also C908.2, C909.2, C910.2, Q901.2 (E), Q902.2 (E), Q903.2 (E), U917.8 (GND); no longer U907.2, U908.2, U909.2, U910.2, U911.2, U912.2, U913.2, U914.2, U915.2, U916.2
- net PA_50MV: now also R948.1; no longer R936.1, R943.1
- net PA_EM: now also R949.1; no longer R945.1
- net PA_MOS1: now also U917.1 (I1); no longer R925.2
- net PA_MOS2: now also U917.2 (I2); no longer R926.2
- net PA_MOS3: now also U917.3 (I3); no longer R927.2
- net PA_MOS4: now also U917.4 (I4); no longer R928.2
- net PA_MOS5: now also U917.5 (I5); no longer R929.2
- net PA_MOS6: now also U917.6 (I6); no longer R930.2
- net PA_NULL: now also R950.1; no longer R947.1
- new net: C908.1, Q901.1 (B), R948.2
- new net: C909.1, Q902.1 (B), R949.2
- new net: C910.1, Q903.1 (B), R950.2
- new net +5VF: R925.2, R926.2, R927.2, R928.2, R929.2, R930.2, R936.1, R943.1, R945.1, R947.1, U917.9 (COM)
- new net 50MV_NPN: Q901.3 (C), U913.2, U914.2
- new net EM_NPN: Q902.3 (C), U915.2
- new net MOS1: U907.2, U917.16 (O1)
- new net MOS2: U908.2, U917.15 (O2)
- new net MOS3: U909.2, U917.14 (O3)
- new net MOS4: U910.2, U917.13 (O4)
- new net MOS5: U911.2, U917.12 (O5)
- new net MOS6: U912.2, U917.11 (O6)
- new net NULL_NPN: Q903.3 (C), U916.2
- no-connect marks 4 -> 6
Other:
- note added: "100"
- note added: "3k01"
- note added: "900"
- moved on the sheet: C901, C902, C903, C904, C905, C906, C907, D901, D902, D903, R901, R902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
