File: hardware/project/ETH1CLCR1/ADC.sch (KiCad schematic (older format))
At the start: 87 parts, among them Q1101 BC847W, Q1102 BC847W, Q1103 BC847W, Q1104 BC847W, U1101 ADG419BR, U1102 ADG419BR, U1103 REF192, U1104 AD8606-2-MSOP, U1105 AD8606-2-MSOP, U1106 AD7380, U1107 AD8605, U1108 LT6350, U1109 LT6350, U1110 OPA602, U1111 OPA602, U1112 PGA103, U1113 PGA103

Commit message: PCB layout
Parts:
- added R1141: 10k, Resistor_SMD:R_0603_1608Metric_Pad1.05x0.95mm_HandSolder, symbol Device:R
- added R1142: 10K, Resistor_SMD:R_0603_1608Metric_Pad1.05x0.95mm_HandSolder, symbol Device:R
- C1108, C1109, C1110, C1113: value 1u -> 100n
Connections:
- net AGNDF: now also R1141.1, R1142.1; no longer U1101.2, U1102.2
- new net: R1141.2, U1102.2
- new net: R1142.2, U1101.2
Other:
- moved on the sheet: C1108, C1109
Changed lines of the file:
@@
 L ETH1CLCR1:AGNDF #PWR01177
 U 1 1 5E0AEDBA
-P 14200 2100
-F 0 "#PWR01177" H 14200 1850 50  0001 C CNN
-F 1 "AGNDF" V 14205 1972 50  0000 R CNN
-F 2 "" H 14200 2100 50  0001 C CNN
-F 3 "" H 14200 2100 50  0001 C CNN
-	1    14200 2100
+P 14550 2100
+F 0 "#PWR01177" H 14550 1850 50  0001 C CNN
+F 1 "AGNDF" V 14555 1972 50  0000 R CNN
+F 2 "" H 14550 2100 50  0001 C CNN
+F 3 "" H 14550 2100 50  0001 C CNN
+	1    14550 2100
 	0    -1   -1   0
 $EndComp
@@
 L ETH1CLCR1:AGNDF #PWR01178
 U 1 1 5E0D67C9
-P 14200 5000
-F 0 "#PWR01178" H 14200 4750 50  0001 C CNN
-F 1 "AGNDF" V 14205 4872 50  0000 R CNN
-F 2 "" H 14200 5000 50  0001 C CNN
-F 3 "" H 14200 5000 50  0001 C CNN
-	1    14200 5000
+P 14550 5000
+F 0 "#PWR01178" H 14550 4750 50  0001 C CNN
+F 1 "AGNDF" V 14555 4872 50  0000 R CNN
+F 2 "" H 14550 5000 50  0001 C CNN
+F 3 "" H 14550 5000 50  0001 C CNN
+	1    14550 5000
 	0    -1   -1   0
 $EndComp
@@
 P 5650 10400
 F 0 "C1110" H 5765 10446 50  0000 L CNN
-F 1 "1u" H 5765 10355 50  0000 L CNN
+F 1 "100n" H 5765 10355 50  0000 L CNN
 F 2 "Capacitor_SMD:C_0603_1608Metric_Pad1.05x0.95mm_HandSolder" H 5688 10250 50  0001 C CNN
 F 3 "~" H 5650 10400 50  0001 C CNN
@@
 P 6150 10400
 F 0 "C1113" H 6265 10446 50  0000 L CNN
-F 1 "1u" H 6265 10355 50  0000 L CNN
+F 1 "100n" H 6265 10355 50  0000 L CNN
 F 2 "Capacitor_SMD:C_0603_1608Metric_Pad1.05x0.95mm_HandSolder" H 6188 10250 50  0001 C CNN
 F 3 "~" H 6150 10400 50  0001 C CNN
@@
 L Device:C C1108
 U 1 1 5ECFACDE
-P 4700 10400
-F 0 "C1108" H 4815 10446 50  0000 L CNN
-F 1 "1u" H 4815 10355 50  0000 L CNN
-F 2 "Capacitor_SMD:C_0603_1608Metric_Pad1.05x0.95mm_HandSolder" H 4738 10250 50  0001 C CNN
-F 3 "~" H 4700 10400 50  0001 C CNN
-	1    4700 10400
+P 4650 10400
+F 0 "C1108" H 4765 10446 50  0000 L CNN
+F 1 "100n" H 4765 10355 50  0000 L CNN
+F 2 "Capacitor_SMD:C_0603_1608Metric_Pad1.05x0.95mm_HandSolder" H 4688 10250 50  0001 C CNN
+F 3 "~" H 4650 10400 50  0001 C CNN
+	1    4650 10400
 	1    0    0    -1
 $EndComp
@@
 L Device:C C1109
 U 1 1 5ECFACE4
-P 5200 10400
-F 0 "C1109" H 5315 10446 50  0000 L CNN
-F 1 "1u" H 5315 10355 50  0000 L CNN
-F 2 "Capacitor_SMD:C_0603_1608Metric_Pad1.05x0.95mm_HandSolder" H 5238 10250 50  0001 C CNN
-F 3 "~" H 5200 10400 50  0001 C CNN
-	1    5200 10400
+P 5150 10400
+F 0 "C1109" H 5265 10446 50  0000 L CNN
+F 1 "100n" H 5265 10355 50  0000 L CNN
+F 2 "Capacitor_SMD:C_0603_1608Metric_Pad1.05x0.95mm_HandSolder" H 5188 10250 50  0001 C CNN
+F 3 "~" H 5150 10400 50  0001 C CNN
+	1    5150 10400
 	1    0    0    -1
 $EndComp
@@
 L ETH1CLCR1:AGNDF #PWR01124
 U 1 1 5ECFACEA
-P 4700 10700
-F 0 "#PWR01124" H 4700 10450 50  0001 C CNN
-F 1 "AGNDF" H 4705 10527 50  0000 C CNN
-F 2 "" H 4700 10700 50  0001 C CNN
-F 3 "" H 4700 10700 50  0001 C CNN
-	1    4700 10700
+P 4650 10700
+F 0 "#PWR01124" H 4650 10450 50  0001 C CNN
+F 1 "AGNDF" H 4655 10527 50  0000 C CNN
+F 2 "" H 4650 10700 50  0001 C CNN
+F 3 "" H 4650 10700 50  0001 C CNN
+	1    4650 10700
 	1    0    0    -1
 $EndComp
@@
 L ETH1CLCR1:AGNDF #PWR01126
 U 1 1 5ECFACF0
-P 5200 10700
-F 0 "#PWR01126" H 5200 10450 50  0001 C CNN
-F 1 "AGNDF" H 5205 10527 50  0000 C CNN
-F 2 "" H 5200 10700 50  0001 C CNN
-F 3 "" H 5200 10700 50  0001 C CNN
-	1    5200 10700
-	1    0    0    -1
-$EndComp
-Wire Wire Line
-	4700 10700 4700 10550
-Wire Wire Line
-	4700 10250 4700 10100
-Wire Wire Line
-	5200 10700 5200 10550
-Wire Wire Line
-	5200 10250 5200 10100
+P 5150 10700
+F 0 "#PWR01126" H 5150 10450 50  0001 C CNN
+F 1 "AGNDF" H 5155 10527 50  0000 C CNN
+F 2 "" H 5150 10700 50  0001 C CNN
+F 3 "" H 5150 10700 50  0001 C CNN
+	1    5150 10700
+	1    0    0    -1
+$EndComp
+Wire Wire Line
+	4650 10700 4650 10550
+Wire Wire Line
+	4650 10250 4650 10100
+Wire Wire Line
+	5150 10700 5150 10550
+Wire Wire Line
+	5150 10250 5150 10100
 $Comp
 L ETH1CLCR1:+3.3VF #PWR01123
 U 1 1 5ECFACFA
-P 4700 10100
-F 0 "#PWR01123" H 4700 9950 50  0001 C CNN
-F 1 "+3.3VF" H 4715 10273 50  0000 C CNN
-F 2 "" H 4700 10100 50  0001 C CNN
-F 3 "" H 4700 10100 50  0001 C CNN
-	1    4700 10100
+P 4650 10100
+F 0 "#PWR01123" H 4650 9950 50  0001 C CNN
+F 1 "+3.3VF" H 4665 10273 50  0000 C CNN
+F 2 "" H 4650 10100 50  0001 C CNN
+F 3 "" H 4650 10100 50  0001 C CNN
+	1    4650 10100
 	1    0    0    -1
 $EndComp
@@
 L ETH1CLCR1:+3.3VF #PWR01125
 U 1 1 5ECFAD00
-P 5200 10100
-F 0 "#PWR01125" H 5200 9950 50  0001 C CNN
-F 1 "+3.3VF" H 5215 10273 50  0000 C CNN
-F 2 "" H 5200 10100 50  0001 C CNN
-F 3 "" H 5200 10100 50  0001 C CNN
-	1    5200 10100
+P 5150 10100
+F 0 "#PWR01125" H 5150 9950 50  0001 C CNN
+F 1 "+3.3VF" H 5165 10273 50  0000 C CNN
+F 2 "" H 5150 10100 50  0001 C CNN
+F 3 "" H 5150 10100 50  0001 C CNN
+	1    5150 10100
 	1    0    0    -1
 $EndComp
@@
 	-1   0    0    -1
 $EndComp
+$Comp
+L Device:R R1141
+U 1 1 5EC59EDC
+P 14350 2100
+F 0 "R1141" V 14143 2100 50  0000 C CNN
+F 1 "10k" V 14234 2100 50  0000 C CNN
+F 2 "Resistor_SMD:R_0603_1608Metric_Pad1.05x0.95mm_HandSolder" V 14280 2100 50  0001 C CNN
+F 3 "~" H 14350 2100 50  0001 C CNN
+	1    14350 2100
+	0    1    1    0
+$EndComp
+Wire Wire Line
+	14550 2100 14500 2100
+$Comp
+L Device:R R1142
+U 1 1 5EC77936
+P 14350 5000
+F 0 "R1142" V 14143 5000 50  0000 C CNN
+F 1 "10K" V 14234 5000 50  0000 C CNN
+F 2 "Resistor_SMD:R_0603_1608Metric_Pad1.05x0.95mm_HandSolder" V 14280 5000 50  0001 C CNN
+F 3 "~" H 14350 5000 50  0001 C CNN
+	1    14350 5000
+	0    1    1    0
+$EndComp
+Wire Wire Line
+	14550 5000 14500 5000
 $EndSCHEMATC
