File: hardware/project/ETH1CLCR1/ADC.sch (KiCad schematic (older format))
At the start: 103 parts, among them Q1101 BC847W, Q1102 BC847W, Q1103 BC847W, Q1104 BC847W, U1101 ADG419BR, U1102 ADG419BR, U1103 ADR4525BRZ, U1104 ADA4807-2ARM, U1106 AD7380, U1106 ADA4807-2ARM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

Commit message: Changed BC847W base resistor from 1k to 10k.
Parts:
- R1139, R1140, R1145, R1146: value 1k -> 10k
Changed lines of the file:
@@
 AR Path="/5E402F62/5E39CEEC" Ref="R1140"  Part="1"
 F 0 "R1140" V 12893 9150 50  0000 C CNN
-F 1 "1k" V 12984 9150 50  0000 C CNN
+F 1 "10k" V 12984 9150 50  0000 C CNN
 F 2 "Resistor_SMD:R_0603_1608Metric_Pad1.05x0.95mm_HandSolder" V 13030 9150 50  0001 C CNN
 F 3 "~" H 13100 9150 50  0001 C CNN
@@
 AR Path="/5E402F62/5E39CF11" Ref="R1139"  Part="1"
 F 0 "R1139" V 12893 7900 50  0000 C CNN
-F 1 "1k" V 12984 7900 50  0000 C CNN
+F 1 "10k" V 12984 7900 50  0000 C CNN
 F 2 "Resistor_SMD:R_0603_1608Metric_Pad1.05x0.95mm_HandSolder" V 13030 7900 50  0001 C CNN
 F 3 "~" H 13100 7900 50  0001 C CNN
@@
 AR Path="/5E402F62/5E39CF36" Ref="R1146"  Part="1"
 F 0 "R1146" V 14943 9150 50  0000 C CNN
-F 1 "1k" V 15034 9150 50  0000 C CNN
+F 1 "10k" V 15034 9150 50  0000 C CNN
 F 2 "Resistor_SMD:R_0603_1608Metric_Pad1.05x0.95mm_HandSolder" V 15080 9150 50  0001 C CNN
 F 3 "~" H 15150 9150 50  0001 C CNN
@@
 AR Path="/5E402F62/5E39CF5B" Ref="R1145"  Part="1"
 F 0 "R1145" V 14943 7900 50  0000 C CNN
-F 1 "1k" V 15034 7900 50  0000 C CNN
+F 1 "10k" V 15034 7900 50  0000 C CNN
 F 2 "Resistor_SMD:R_0603_1608Metric_Pad1.05x0.95mm_HandSolder" V 15080 7900 50  0001 C CNN
 F 3 "~" H 15150 7900 50  0001 C CNN

Commit message: Small changes in schematics and PCB
Parts:
- R1121, R1122, R1125, R1127: value 12k -> 12k/.1%
- R1123, R1124, R1129, R1130: value 52k3 -> 52k3/.1%
- R1126, R1128: value 10k -> 10k/.1%
Other:
- moved on the sheet: R1129, R1130
Changed lines of the file:
@@
 L Device:R R1129
 U 1 1 5E3FB300
-P 10650 2200
-F 0 "R1129" V 10443 2200 50  0000 C CNN
-F 1 "52k3" V 10534 2200 50  0000 C CNN
-F 2 "Resistor_SMD:R_0603_1608Metric_Pad1.05x0.95mm_HandSolder" V 10580 2200 50  0001 C CNN
-F 3 "~" H 10650 2200 50  0001 C CNN
-	1    10650 2200
+P 10850 2200
+F 0 "R1129" V 10643 2200 50  0000 C CNN
+F 1 "52k3/.1%" V 10734 2200 50  0000 C CNN
+F 2 "Resistor_SMD:R_0603_1608Metric_Pad1.05x0.95mm_HandSolder" V 10780 2200 50  0001 C CNN
+F 3 "~" H 10850 2200 50  0001 C CNN
+	1    10850 2200
 	0    1    1    0
 $EndComp
 Wire Wire Line
-	10800 2200 11850 2200
+	11000 2200 11850 2200
 $Comp
 L Device:R R1126
@@
 P 10200 2400
 F 0 "R1126" H 10270 2446 50  0000 L CNN
-F 1 "10k" H 10270 2355 50  0000 L CNN
+F 1 "10k/.1%" H 10270 2355 50  0000 L CNN
 F 2 "Resistor_SMD:R_0603_1608Metric_Pad1.05x0.95mm_HandSolder" V 10130 2400 50  0001 C CNN
 F 3 "~" H 10200 2400 50  0001 C CNN
@@
 Connection ~ 10200 2200
 Wire Wire Line
-	10200 2200 10500 2200
+	10200 2200 10700 2200
 $Comp
 L ETH1CLCR1:AGNDF #PWR01168
@@
 P 10200 2000
 F 0 "R1125" H 10270 2046 50  0000 L CNN
-F 1 "12k" H 10270 1955 50  0000 L CNN
+F 1 "12k/.1%" H 10270 1955 50  0000 L CNN
 F 2 "Resistor_SMD:R_0603_1608Metric_Pad1.05x0.95mm_HandSolder" V 10130 2000 50  0001 C CNN
 F 3 "~" H 10200 2000 50  0001 C CNN
@@
 P 9550 1550
 F 0 "R1121" V 9343 1550 50  0000 C CNN
-F 1 "12k" V 9434 1550 50  0000 C CNN
+F 1 "12k/.1%" V 9434 1550 50  0000 C CNN
 F 2 "Resistor_SMD:R_0603_1608Metric_Pad1.05x0.95mm_HandSolder" V 9480 1550 50  0001 C CNN
 F 3 "~" H 9550 1550 50  0001 C CNN
@@
 P 10150 1550
 F 0 "R1123" V 9943 1550 50  0000 C CNN
-F 1 "52k3" V 10034 1550 50  0000 C CNN
+F 1 "52k3/.1%" V 10034 1550 50  0000 C CNN
 F 2 "Resistor_SMD:R_0603_1608Metric_Pad1.05x0.95mm_HandSolder" V 10080 1550 50  0001 C CNN
 F 3 "~" H 10150 1550 50  0001 C CNN
@@
 	10000 1550 9950 1550
 Wire Wire Line
-	10800 5100 11850 5100
+	11000 5100 11850 5100
 Connection ~ 9200 5000
 Wire Wire Line
@@
 P 10150 4450
 F 0 "R1124" V 9943 4450 50  0000 C CNN
-F 1 "52k3" V 10034 4450 50  0000 C CNN
+F 1 "52k3/.1%" V 10034 4450 50  0000 C CNN
 F 2 "Resistor_SMD:R_0603_1608Metric_Pad1.05x0.95mm_HandSolder" V 10080 4450 50  0001 C CNN
 F 3 "~" H 10150 4450 50  0001 C CNN
@@
 P 9550 4450
 F 0 "R1122" V 9343 4450 50  0000 C CNN
-F 1 "12k" V 9434 4450 50  0000 C CNN
+F 1 "12k/.1%" V 9434 4450 50  0000 C CNN
 F 2 "Resistor_SMD:R_0603_1608Metric_Pad1.05x0.95mm_HandSolder" V 9480 4450 50  0001 C CNN
 F 3 "~" H 9550 4450 50  0001 C CNN
@@
 P 10200 4900
 F 0 "R1127" H 10270 4946 50  0000 L CNN
-F 1 "12k" H 10270 4855 50  0000 L CNN
+F 1 "12k/.1%" H 10270 4855 50  0000 L CNN
 F 2 "Resistor_SMD:R_0603_1608Metric_Pad1.05x0.95mm_HandSolder" V 10130 4900 50  0001 C CNN
 F 3 "~" H 10200 4900 50  0001 C CNN
@@
 $EndComp
 Wire Wire Line
-	10200 5100 10500 5100
+	10200 5100 10700 5100
 Connection ~ 10200 5100
 Wire Wire Line
@@
 P 10200 5300
 F 0 "R1128" H 10270 5346 50  0000 L CNN
-F 1 "10k" H 10270 5255 50  0000 L CNN
+F 1 "10k/.1%" H 10270 5255 50  0000 L CNN
 F 2 "Resistor_SMD:R_0603_1608Metric_Pad1.05x0.95mm_HandSolder" V 10130 5300 50  0001 C CNN
 F 3 "~" H 10200 5300 50  0001 C CNN
@@
 L Device:R R1130
 U 1 1 5E4A997A
-P 10650 5100
-F 0 "R1130" V 10443 5100 50  0000 C CNN
-F 1 "52k3" V 10534 5100 50  0000 C CNN
-F 2 "Resistor_SMD:R_0603_1608Metric_Pad1.05x0.95mm_HandSolder" V 10580 5100 50  0001 C CNN
-F 3 "~" H 10650 5100 50  0001 C CNN
-	1    10650 5100
+P 10850 5100
+F 0 "R1130" V 10643 5100 50  0000 C CNN
+F 1 "52k3/.1%" V 10734 5100 50  0000 C CNN
+F 2 "Resistor_SMD:R_0603_1608Metric_Pad1.05x0.95mm_HandSolder" V 10780 5100 50  0001 C CNN
+F 3 "~" H 10850 5100 50  0001 C CNN
+	1    10850 5100
 	0    1    1    0
 $EndComp

Commit message: Software development
Parts:
- C1123, C1124: value 1n -> DNP
- R1119, R1120: value 100 -> 0
Changed lines of the file:
@@
 P 8550 2250
 F 0 "C1123" H 8665 2296 50  0000 L CNN
-F 1 "1n" H 8665 2205 50  0000 L CNN
+F 1 "DNP" H 8665 2205 50  0000 L CNN
 F 2 "Capacitor_SMD:C_0603_1608Metric_Pad1.05x0.95mm_HandSolder" H 8588 2100 50  0001 C CNN
 F 3 "~" H 8550 2250 50  0001 C CNN
@@
 P 9000 2100
 F 0 "R1119" V 8793 2100 50  0000 C CNN
-F 1 "100" V 8884 2100 50  0000 C CNN
+F 1 "0" V 8884 2100 50  0000 C CNN
 F 2 "Resistor_SMD:R_0603_1608Metric_Pad1.05x0.95mm_HandSolder" V 8930 2100 50  0001 C CNN
 F 3 "~" H 9000 2100 50  0001 C CNN
@@
 P 9000 5000
 F 0 "R1120" V 8793 5000 50  0000 C CNN
-F 1 "100" V 8884 5000 50  0000 C CNN
+F 1 "0" V 8884 5000 50  0000 C CNN
 F 2 "Resistor_SMD:R_0603_1608Metric_Pad1.05x0.95mm_HandSolder" V 8930 5000 50  0001 C CNN
 F 3 "~" H 9000 5000 50  0001 C CNN
@@
 P 8600 5150
 F 0 "C1124" H 8715 5196 50  0000 L CNN
-F 1 "1n" H 8715 5105 50  0000 L CNN
+F 1 "DNP" H 8715 5105 50  0000 L CNN
 F 2 "Capacitor_SMD:C_0603_1608Metric_Pad1.05x0.95mm_HandSolder" H 8638 5000 50  0001 C CNN
 F 3 "~" H 8600 5150 50  0001 C CNN
