File: hardware/project/ETH1CLCR1/MCU2.sch (KiCad schematic (older format))
At the start: 29 parts, among them J1301 20021111-00010T4LF, U1301 STM32H743ZI, U1302 24LC08B-E/MS, Y1301 NX3225GD-8MHZ-STD-CRA-3

Commit message: PCB layout
Parts:
- added C1320: 100n, Capacitor_SMD:C_0603_1608Metric_Pad1.05x0.95mm_HandSolder, symbol Device:C
- renumbered C1319 to C1305, C1305 to C1306, C1306 to C1307, C1307 to C1308, C1308 to C1309, C1309 to C1310, C1310 to C1311, C1311 to C1312, C1312 to C1313, C1313 to C1314, C1314 to C1315, C1315 to C1316, C1316 to C1317, C1317 to C1318, C1318 to C1319, C1320 to C1321
Connections:
- net +3.3VP: now also C1320.1
- net ADC_NULL1: now also U1301.119 (PD5,USART2_TX,FMC_NWE,EVENTOUT); no longer U1301.140 (PB9,I2C4_SDA,TIM4_CH4,TIM11_CH1,I2C1_SDA,SPI2_NSS,I2S2_WS,DFSDM1_DATIN7,UART5_TX,CAN1_TX,SDMMC2_D5,I2C4_SMBA,SDMMC1_D5,DCMI_D7,LCD_B7,EVENTOUT)
- net ADC_NULL2: now also U1301.122 (PD6,DFSDM1_CKIN4,SPI3_MOSI,I2S3_SD,SAI1_SD_A,USART2_RX,DFSDM1_DATIN1,SDMMC2_CK,FMC_NWAIT,DCMI_D10,LCD_B2,EVENTOUT); no longer U1301.139 (PB8,I2C4_SCL,TIM4_CH3,TIM10_CH1,I2C1_SCL,DFSDM1_CKIN7,UART5_RX,CAN1_RX,SDMMC2_D4,ETH_MII_TXD3,SDMMC1_D4,DCMI_D6,LCD_B6,EVENTOUT)
- net ADC_SCLK: now also U1301.111 (PC10,DFSDM1_CKIN5,SPI3_SCK,I2S3_CK,USART3_TX,UART4_TX,QUADSPI_BK1_IO1,SDMMC1_D2,DCMI_D8,LCD_R2,EVENTOUT); no longer U1301.41 (PA5,TIM2_CH1,TIM2_ETR,TIM8_CH1N,SPI1_SCK,I2S1_CK,SPI6_SCK,OTG_HS_ULPI_CK,LCD_R4,EVENTOUT,ADC1_IN5,ADC2_IN5,DAC_OUT2)
- net ADC_SDI: now also U1301.113 (PC12,TRACED3,SPI3_MOSI,I2S3_SD,USART3_CK,UART5_TX,SDMMC1_CK,DCMI_D9,EVENTOUT); no longer U1301.43 (PA7,TIM1_CH1N,TIM3_CH2,TIM8_CH1N,SPI1_MOSI,I2S1_SD,SPI6_MOSI,TIM14_CH1,ETH_MII_RX_DV,ETH_RMII_CRS_DV,FMC_SDNWE,EVENTOUT,ADC1_IN7,ADC2_IN7)
- net ADC_SDOA: now also U1301.112 (PC11,DFSDM1_DATIN5,SPI3_MISO,USART3_RX,UART4_RX,QUADSPI_BK2_NCS,SDMMC1_D3,DCMI_D4,EVENTOUT); no longer U1301.42 (PA6,TIM1_BKIN,TIM3_CH1,TIM8_BKIN,SPI1_MISO,SPI6_MISO,TIM13_CH1,MDIOS_MDC,DCMI_PIXCLK,LCD_G2,EVENTOUT,ADC1_IN6,ADC2_IN6)
- net ADC_~ALARM: now also U1301.114 (PD0,DFSDM1_CKIN6,DFSDM1_DATIN7,UART4_RX,CAN1_RX,FMC_D2,EVENTOUT); no longer U1301.37 (PA3,TIM2_CH4,TIM5_CH4,TIM9_CH2,USART2_RX,LCD_B2,OTG_HS_ULPI_D0,ETH_MII_COL,LCD_B5,EVENTOUT,ADC1_IN3,ADC2_IN3,ADC3_IN3)
- net ADC_~CS: now also U1301.110 (PA15,JTDI,TIM2_CH1,TIM2_ETR,HDMI_CEC,SPI1_NSS,I2S1_WS,SPI3_NSS,I2S3_WS,SPI6_NSS,UART4_RTS,CAN3_TX,UART7_TX,EVENTOUT); no longer U1301.40 (PA4,SPI1_NSS,I2S1_WS,SPI3_NSS,I2S3_WS,USART2_CK,SPI6_NSS,OTG_HS_SOF,DCMI_HSYNC,LCD_VSYNC,EVENTOUT,ADC1_IN4,ADC2_IN4,DAC_OUT1)
- net CXN_REL1: now also U1301.63 (PE10,TIM1_CH2N,DFSDM1_DATIN4,UART7_CTS,QUADSPI_BK2_IO3,FMC_D7,EVENTOUT); no longer U1301.49 (PF11,SAI1_SD_A,SPI3_MOSI,I2S3_SD,QUADSPI_CLK,DFSDM1_CKIN1,EVENTOUT)
- net CXN_REL2: now also U1301.60 (PE9,TIM1_CH1,DFSDM1_CKOUT,UART7_RTS,QUADSPI_BK2_IO2,FMC_D6,EVENTOUT); no longer U1301.48 (PB2,SAI1_SD_A,SPI3_MOSI,I2S3_SD,QUADSPI_CLK,DFSDM1_CKIN1,EVENTOUT)
- net CXN_REL3: now also U1301.59 (PE8,TIM1_CH1N,DFSDM1_CKIN2,UART7_TX,QUADSPI_BK2_IO1,FMC_D5,EVENTOUT); no longer U1301.47 (PB1,TIM1_CH3N,TIM3_CH4,TIM8_CH3N,DFSDM1_DATIN1,LCD_R6,OTG_HS_ULPI_D2,ETH_MII_RXD3,LCD_G0,EVENTOUT,ADC1_IN9,ADC2_IN9)
- net CXN_REL4: now also U1301.58 (PE7,TIM1_ETR,DFSDM1_DATIN2,UART7_RX,QUADSPI_BK2_IO0,FMC_D4,EVENTOUT); no longer U1301.46 (PB0,TIM1_CH2N,TIM3_CH3,TIM8_CH2N,DFSDM1_CKOUT,UART4_CTS,_LCD_R3,OTG_HS_ULPI_D1,ETH_MII_RXD2,LCD_G1,EVENTOUT,ADC1_IN8,ADC2_IN8)
- net CXN_REL5: now also U1301.57 (PG1,FMC_A11,EVENTOUT); no longer U1301.45 (PC5,DFSDM1_DATIN2,SPDIF_RX3,ETH_MII_RXD1,ETH_RMII_RXD1,FMC_SDCKE0,EVENTOUT,ADC1_IN15,ADC2_IN15)
- net CXN_REL6: now also U1301.56 (PG0,FMC_A10,EVENTOUT); no longer U1301.44 (PC4,DFSDM1_CKIN2,I2S1_MCK,SPDIF_RX2,ETH_MII_RXD0,ETH_RMII_RXD0,FMC_SDNE0,EVENTOUT,ADC1_IN14,ADC2_IN14)
- net DAC_~CLR: now also U1301.15 (PF5,FMC_A5,EVENTOUT,ADC3_IN15); no longer U1301.14 (PF4,FMC_A4,EVENTOUT,ADC3_IN14)
- net DAC_~LDAC: now also U1301.14 (PF4,FMC_A4,EVENTOUT,ADC3_IN14); no longer U1301.15 (PF5,FMC_A5,EVENTOUT,ADC3_IN15)
- net DGNDF: now also C1320.2
- net FB_CAP: now also U1301.69 (PB10,TIM2_CH3,I2C2_SCL,SPI2_SCK,I2S2_CK,DFSDM1_DATIN7,USART3_TX,QUADSPI_BK1_NCS,OTG_HS_ULPI_D3,ETH_MII_RX_ER,LCD_G4,EVENTOUT); no longer U1301.124 (PG9,SPI1_MISO,SPDIF_RX3,USART6_RX,QUADSPI_BK2_IO2,SAI2_FS_B,SDMMC2_D0,FMC_NE2,FMC_NCE,DCMI_VSYNC,EVENTOUT)
- net FB_CLK: now also U1301.74 (PB13,TIM1_CH1N,SPI2_SCK,I2S2_CK,DFSDM1_CKIN1,USART3_CTS,UART5_TX,CAN2_TX,OTG_HS_ULPI_D6,ETH_MII_TXD1,ETH_RMII_TXD1,EVENTOUT,OTG_HS_VBUS); no longer U1301.128 (PG13,TRACED0,LPTIM1_OUT,SPI6_SCK,USART6_CTS,ETH_MII_TXD0,ETH_RMII_TXD0,FMC_A24,LCD_R0,EVENTOUT)
- net FB_RDY: now also U1301.78 (PD9,DFSDM1_DATIN3,USART3_RX,FMC_D14,EVENTOUT); no longer U1301.125 (PG10,SPI1_NSS,I2S1_WS,LCD_G3,SAI2_SD_B,SDMMC2_D1,FMC_NE3,DCMI_D2,LCD_B2,EVENTOUT)
- net FB_SDI: now also U1301.76 (PB15,RTC_REFIN,TIM1_CH3N,TIM8_CH3N,USART1_RX,SPI2_MOSI,I2S2_SD,DFSDM1_CKIN2,UART4_CTS,TIM12_CH2,SDMMC2_D1,OTG_HS_DP,EVENTOUT); no longer U1301.129 (PG14,TRACED1,LPTIM1_ETR,SPI6_MOSI,USART6_TX,QUADSPI_BK2_IO3,ETH_MII_TXD1,ETH_RMII_TXD1,FMC_A25,LCD_B0,EVENTOUT)
- net FB_SDO: now also U1301.75 (PB14,TIM1_CH2N,TIM8_CH2N,USART1_TX,SPI2_MISO,DFSDM1_DATIN2,USART3_RTS,UART4_RTS,TIM12_CH1,SDMMC2_D0,OTG_HS_DM,EVENTOUT); no longer U1301.127 (PG12,LPTIM1_IN1,SPI6_MISO,SPDIF_RX1,USART6_RTS,LCD_B4,SDMMC2_D3,FMC_NE4,LCD_B1,EVENTOUT)
- net FB_~CS: now also U1301.73 (PB12,TIM1_BKIN,I2C2_SMBA,SPI2_NSS,I2S2_WS,DFSDM1_DATIN1,USART3_CK,UART5_RX,CAN2_RX,OTG_HS_ULPI_D5,ETH_MII_TXD0,ETH_RMII_TXD0,OTG_HS_ID,EVENTOUT); no longer U1301.93 (PG8,SPI6_NSS,SPDIF_RX2,USART6_RTS,ETH_PPS_OUT,FMC_SDCLK,LCD_G7,EVENTOUT)
- net FB_~RST: now also U1301.79 (PD10,DFSDM1_CKOUT,USART3_CK,FMC_D15,LCD_B3,EVENTOUT); no longer U1301.126 (PG11,SPI1_SCK,I2S1_CK,SPDIF_RX0,SDMMC2_D2,ETH_MII_TX_EN,ETH_RMII_TX_EN,DCMI_D3,LCD_B3,EVENTOUT)
- net G1A0_CTR: now also U1301.116 (PD2,TRACED2,TIM3_ETR,UART5_RX,SDMMC1_CMD,DCMI_D11,EVENTOUT); no longer U1301.135 (PB5,UART5_RX,TIM3_CH2,I2C1_SMBA,SPI1_MOSI,I2S1_SD,SPI3_MOSI,I2S3_SD,SPI6_MOSI,CAN2_RX,OTG_HS_ULPI_D7,ETH_PPS_OUT,FMC_SDCKE1,DCMI_D10,LCD_G7,EVENTOUT)
- net G1A1_CTR: now also U1301.115 (PD1,DFSDM1_DATIN6,DFSDM1_CKIN7,UART4_TX,CAN1_TX,FMC_D3,EVENTOUT); no longer U1301.134 (PB4,NJTRST,TIM3_CH1,SPI1_MISO,SPI3_MISO,SPI2_NSS,I2S2_WS,SPI6_MISO,SDMMC2_D3,CAN3_TX,UART7_TX,EVENTOUT)
- net G2A0_CTR: now also U1301.118 (PD4,DFSDM1_CKIN0,USART2_RTS,FMC_NOE,EVENTOUT); no longer U1301.137 (PB7,TIM4_CH2,I2C1_SDA,DFSDM1_CKIN5,USART1_RX,I2C4_SDA,FMC_NL,DCMI_VSYNC,EVENTOUT)
- net G2A1_CTR: now also U1301.117 (PD3,DFSDM1_CKOUT,SPI2_SCK,I2S2_CK,DFSDM1_DATIN0,USART2_CTS,FMC_CLK,DCMI_D5,LCD_G7,EVENTOUT); no longer U1301.136 (PB6,UART5_TX,TIM4_CH1,HDMI_CEC,I2C1_SCL,DFSDM1_DATIN5,USART1_TX,CAN2_TX,QUADSPI_BK1_NCS,I2C4_SCL,FMC_SDNE1,DCMI_D5,EVENTOUT)
- net MCU1_GPIO_OUT1: now also U1301.47 (PB1,TIM1_CH3N,TIM3_CH4,TIM8_CH3N,DFSDM1_DATIN1,LCD_R6,OTG_HS_ULPI_D2,ETH_MII_RXD3,LCD_G0,EVENTOUT,ADC1_IN9,ADC2_IN9); no longer U1301.7 (PC13,EVENTOUT,RTC_TAMP2,RTC_TS,WKUP5)
- net MCU1_GPIO_OUT2: now also U1301.48 (PB2,SAI1_SD_A,SPI3_MOSI,I2S3_SD,QUADSPI_CLK,DFSDM1_CKIN1,EVENTOUT); no longer U1301.8 (PC14,EVENTOUT,OSC32_IN)
- net MCU1_MISO: now also U1301.42 (PA6,TIM1_BKIN,TIM3_CH1,TIM8_BKIN,SPI1_MISO,SPI6_MISO,TIM13_CH1,MDIOS_MDC,DCMI_PIXCLK,LCD_G2,EVENTOUT,ADC1_IN6,ADC2_IN6); no longer U1301.4 (PE5,TRACED2,TIM9_CH1,SPI4_MISO,SAI1_SCK_A,DFSDM1_CKIN3,FMC_A21,DCMI_D6,LCD_G0,EVENTOUT)
- net MCU1_MOSI: now also U1301.43 (PA7,TIM1_CH1N,TIM3_CH2,TIM8_CH1N,SPI1_MOSI,I2S1_SD,SPI6_MOSI,TIM14_CH1,ETH_MII_RX_DV,ETH_RMII_CRS_DV,FMC_SDNWE,EVENTOUT,ADC1_IN7,ADC2_IN7); no longer U1301.5 (PE6,TRACED3,TIM1_BKIN2,TIM9_CH2,SPI4_MOSI,SAI1_SD_A,SAI2_MCLK_B,FMC_A22,DCMI_D7,LCD_G1,EVENTOUT)
- net MCU1_SCLK: now also U1301.41 (PA5,TIM2_CH1,TIM2_ETR,TIM8_CH1N,SPI1_SCK,I2S1_CK,SPI6_SCK,OTG_HS_ULPI_CK,LCD_R4,EVENTOUT,ADC1_IN5,ADC2_IN5,DAC_OUT2); no longer U1301.1 (PE2,TRACECLK,SPI4_SCK,SAI1_MCLK_A,QUADSPI_BK1_IO2,ETH_MII_TXD3,FMC_A23,EVENTOUT)
- net MCU1_STATUS_IN1: now also U1301.49 (PF11,SAI1_SD_A,SPI3_MOSI,I2S3_SD,QUADSPI_CLK,DFSDM1_CKIN1,EVENTOUT); no longer U1301.9 (PC15,EVENTOUT,OSC32_OUT)
- net MCU1_STATUS_IN2: now also U1301.50 (PF12,FMC_A6,EVENTOUT); no longer U1301.10 (PF0,I2C2_SDA,FMC_A0,EVENTOUT)
- net MCU1_~SS: now also U1301.40 (PA4,SPI1_NSS,I2S1_WS,SPI3_NSS,I2S3_WS,USART2_CK,SPI6_NSS,OTG_HS_SOF,DCMI_HSYNC,LCD_VSYNC,EVENTOUT,ADC1_IN4,ADC2_IN4,DAC_OUT1); no longer U1301.3 (PE4,TRACED1,SPI4_NSS,SAI1_FS_A,DFSDM1_DATIN3,FMC_A20,DCMI_D4,LCD_B0,EVENTOUT)
- net MCU3_MISO: now also U1301.4 (PE5,TRACED2,TIM9_CH1,SPI4_MISO,SAI1_SCK_A,DFSDM1_CKIN3,FMC_A21,DCMI_D6,LCD_G0,EVENTOUT); no longer U1301.112 (PC11,DFSDM1_DATIN5,SPI3_MISO,USART3_RX,UART4_RX,QUADSPI_BK2_NCS,SDMMC1_D3,DCMI_D4,EVENTOUT)
- net MCU3_MOSI: now also U1301.5 (PE6,TRACED3,TIM1_BKIN2,TIM9_CH2,SPI4_MOSI,SAI1_SD_A,SAI2_MCLK_B,FMC_A22,DCMI_D7,LCD_G1,EVENTOUT); no longer U1301.113 (PC12,TRACED3,SPI3_MOSI,I2S3_SD,USART3_CK,UART5_TX,SDMMC1_CK,DCMI_D9,EVENTOUT)
- net MCU3_NSS: now also U1301.3 (PE4,TRACED1,SPI4_NSS,SAI1_FS_A,DFSDM1_DATIN3,FMC_A20,DCMI_D4,LCD_B0,EVENTOUT); no longer U1301.110 (PA15,JTDI,TIM2_CH1,TIM2_ETR,HDMI_CEC,SPI1_NSS,I2S1_WS,SPI3_NSS,I2S3_WS,SPI6_NSS,UART4_RTS,CAN3_TX,UART7_TX,EVENTOUT)
- net MCU3_SCLK: now also U1301.1 (PE2,TRACECLK,SPI4_SCK,SAI1_MCLK_A,QUADSPI_BK1_IO2,ETH_MII_TXD3,FMC_A23,EVENTOUT); no longer U1301.111 (PC10,DFSDM1_CKIN5,SPI3_SCK,I2S3_CK,USART3_TX,UART4_TX,QUADSPI_BK1_IO1,SDMMC1_D2,DCMI_D8,LCD_R2,EVENTOUT)
- net PA_50MV: now also U1301.104 (PA12,TIM1_ETR,SPI2_SCK,I2S2_CK,UART4_TX,USART1_RTS,SAI2_FS_B,CAN1_TX,OTG_FS_DP,LCD_R5,EVENTOUT); no longer U1301.60 (PE9,TIM1_CH1,DFSDM1_CKOUT,UART7_RTS,QUADSPI_BK2_IO2,FMC_D6,EVENTOUT)
- net PA_EM: now also U1301.103 (PA11,TIM1_CH4,SPI2_NSS,I2S2_WS,UART4_RX,USART1_CTS,CAN1_RX,OTG_FS_DM,LCD_R4,EVENTOUT); no longer U1301.59 (PE8,TIM1_CH1N,DFSDM1_CKIN2,UART7_TX,QUADSPI_BK2_IO1,FMC_D5,EVENTOUT)
- net PA_ER: now also U1301.102 (PA10,TIM1_CH3,USART1_RX,LCD_B4,OTG_FS_ID,MDIOS_MDIO,DCMI_D1,LCD_B1,EVENTOUT); no longer U1301.58 (PE7,TIM1_ETR,DFSDM1_DATIN2,UART7_RX,QUADSPI_BK2_IO0,FMC_D4,EVENTOUT)
- net PA_MOS1: now also U1301.97 (PC7,TIM3_CH2,TIM8_CH2,I2S3_MCK,DFSDM1_DATIN3,USART6_RX,FMC_NE1,SDMMC2_D7,SDMMC1_D7,DCMI_D1,LCD_G6,EVENTOUT); no longer U1301.63 (PE10,TIM1_CH2N,DFSDM1_DATIN4,UART7_CTS,QUADSPI_BK2_IO3,FMC_D7,EVENTOUT)
- net PA_MOS2: now also U1301.96 (PC6,TIM3_CH1,TIM8_CH1,I2S2_MCK,DFSDM1_CKIN3,USART6_TX,FMC_NWAIT,SDMMC2_D6,SDMMC1_D6,DCMI_D0,LCD_HSYNC,EVENTOUT); no longer U1301.64 (PE11,TIM1_CH2,SPI4_NSS,DFSDM1_CKIN4,SAI2_SD_B,FMC_D8,LCD_G3,EVENTOUT)
- net PA_MOS3: now also U1301.99 (PC9,MCO2,TIM3_CH4,TIM8_CH4,I2C3_SDA,I2S_CKIN,UART5_CTS,QUADSPI_BK1_IO0,LCD_G3,SDMMC1_D1,DCMI_D3,LCD_B2,EVENTOUT); no longer U1301.65 (PE12,TIM1_CH3N,SPI4_SCK,DFSDM1_DATIN5,SAI2_SCK_B,FMC_D9,LCD_B4,EVENTOUT)
- net PA_MOS4: now also U1301.98 (PC8,TRACED1,TIM3_CH3,TIM8_CH3,UART5_RTS,USART6_CK,FMC_NE2,FMC_NCE,SDMMC1_D0,DCMI_D2,EVENTOUT); no longer U1301.66 (PE13,TIM1_CH3,SPI4_MISO,DFSDM1_CKIN5,SAI2_FS_B,FMC_D10,LCD_DE,EVENTOUT)
- net PA_MOS5: now also U1301.101 (PA9,TIM1_CH2,I2C3_SMBA,SPI2_SCK,I2S2_CK,USART1_TX,DCMI_D0,LCD_R5,EVENTOUT,OTG_FS_VBUS); no longer U1301.67 (PE14,TIM1_CH4,SPI4_MOSI,SAI2_MCLK_B,FMC_D11,LCD_CLK,EVENTOUT)
- net PA_MOS6: now also U1301.100 (PA8,MCO1,TIM1_CH1,TIM8_BKIN2,I2C3_SCL,USART1_CK,OTG_FS_SOF,CAN3_RX,UART7_RX,LCD_B3,LCD_R6,EVENTOUT); no longer U1301.68 (PE15,TIM1_BKIN,FMC_D12,LCD_R7,EVENTOUT)
- net RR_100CRT: now also U1301.86 (PD15,TIM4_CH4,UART8_RTS,FMC_D1,EVENTOUT); no longer U1301.79 (PD10,DFSDM1_CKOUT,USART3_CK,FMC_D15,LCD_B3,EVENTOUT)
- net RR_100KCRT: now also U1301.89 (PG4,FMC_A14,FMC_BA0,EVENTOUT); no longer U1301.82 (PD13,TIM4_CH2,LPTIM1_OUT,I2C4_SDA,QUADSPI_BK1_IO3,SAI2_SCK_A,FMC_A18,EVENTOUT)
- net RR_10CRT: now also U1301.85 (PD14,TIM4_CH3,UART8_CTS,FMC_D0,EVENTOUT); no longer U1301.78 (PD9,DFSDM1_DATIN3,USART3_RX,FMC_D14,EVENTOUT)
- net RR_10KCRT: now also U1301.88 (PG3,FMC_A13,EVENTOUT); no longer U1301.81 (PD12,TIM4_CH1,LPTIM1_IN1,I2C4_SCL,USART3_RTS,QUADSPI_BK1_IO1,SAI2_FS_A,FMC_A17,FMC_ALE,EVENTOUT)
- net RR_1KCRT: now also U1301.87 (PG2,FMC_A12,EVENTOUT); no longer U1301.80 (PD11,I2C4_SMBA,USART3_CTS,QUADSPI_BK1_IO0,SAI2_SD_A,FMC_A16,FMC_CLE,EVENTOUT)
- net RR_CLK: now also U1301.126 (PG11,SPI1_SCK,I2S1_CK,SPDIF_RX0,SDMMC2_D2,ETH_MII_TX_EN,ETH_RMII_TX_EN,DCMI_D3,LCD_B3,EVENTOUT); no longer U1301.69 (PB10,TIM2_CH3,I2C2_SCL,SPI2_SCK,I2S2_CK,DFSDM1_DATIN7,USART3_TX,QUADSPI_BK1_NCS,OTG_HS_ULPI_D3,ETH_MII_RX_ER,LCD_G4,EVENTOUT)
- net RR_HA3-COMP: now also U1301.82 (PD13,TIM4_CH2,LPTIM1_OUT,I2C4_SDA,QUADSPI_BK1_IO3,SAI2_SCK_A,FMC_A18,EVENTOUT); no longer U1301.86 (PD15,TIM4_CH4,UART8_RTS,FMC_D1,EVENTOUT)
- net RR_RDY: now also U1301.127 (PG12,LPTIM1_IN1,SPI6_MISO,SPDIF_RX1,USART6_RTS,LCD_B4,SDMMC2_D3,FMC_NE4,LCD_B1,EVENTOUT); no longer U1301.26 (PC0,DFSDM1_CKIN0,DFSDM1_DATIN4,SAI2_FS_B,OTG_HS_ULPI_STP,FMC_SDNWE,LCD_R5,EVENTOUT,ADC1_IN10,ADC2_IN10,ADC3_IN10)
- net RR_RELAYCTR: now also U1301.81 (PD12,TIM4_CH1,LPTIM1_IN1,I2C4_SCL,USART3_RTS,QUADSPI_BK1_IO1,SAI2_FS_A,FMC_A17,FMC_ALE,EVENTOUT); no longer U1301.85 (PD14,TIM4_CH3,UART8_CTS,FMC_D0,EVENTOUT)
- net RR_SDI: now also U1301.123 (PD7,DFSDM1_DATIN4,SPI1_MOSI,I2S1_SD,DFSDM1_CKIN1,USART2_CK,SPDIF_RX0,SDMMC2_CMD,FMC_NE1,EVENTOUT); no longer U1301.27 (PC1,TRACED0,_DFSDM1_DATIN0,SPI2_MOSI,I2S2_SD,SAI1_SD_A,DFSDM1_CKIN4,ETH_MDC,MDIOS_MDC,EVENTOUT,ADC1_IN11,ADC2_IN11,ADC3_IN11,RTC_TAMP3,WKUP3)
- net RR_SDO: now also U1301.124 (PG9,SPI1_MISO,SPDIF_RX3,USART6_RX,QUADSPI_BK2_IO2,SAI2_FS_B,SDMMC2_D0,FMC_NE2,FMC_NCE,DCMI_VSYNC,EVENTOUT); no longer U1301.28 (PC2,DFSDM1_CKIN1,SPI2_MISO,DFSDM1_CKOUT,OTG_HS_ULPI_DIR,ETH_MII_TXD2,FMC_SDNE0,EVENTOUT,ADC1_IN12,ADC2_IN12,ADC3_IN12)
- net RR_~CS: now also U1301.125 (PG10,SPI1_NSS,I2S1_WS,LCD_G3,SAI2_SD_B,SDMMC2_D1,FMC_NE3,DCMI_D2,LCD_B2,EVENTOUT); no longer U1301.73 (PB12,TIM1_BKIN,I2C2_SMBA,SPI2_NSS,I2S2_WS,DFSDM1_DATIN1,USART3_CK,UART5_RX,CAN2_RX,OTG_HS_ULPI_D5,ETH_MII_TXD0,ETH_RMII_TXD0,OTG_HS_ID,EVENTOUT)
- net RR_~RST: now also U1301.128 (PG13,TRACED0,LPTIM1_OUT,SPI6_SCK,USART6_CTS,ETH_MII_TXD0,ETH_RMII_TXD0,FMC_A24,LCD_R0,EVENTOUT); no longer U1301.29 (PC3,DFSDM1_DATIN1,SPI2_MOSI,I2S2_SD,OTG_HS_ULPI_NXT,ETH_MII_TX_CLK,FMC_SDCKE0,EVENTOUT,ADC1_IN13,ADC2_IN13,ADC3_IN13)
- net SR_100CTR: now also U1301.66 (PE13,TIM1_CH3,SPI4_MISO,DFSDM1_CKIN5,SAI2_FS_B,FMC_D10,LCD_DE,EVENTOUT); no longer U1301.122 (PD6,DFSDM1_CKIN4,SPI3_MOSI,I2S3_SD,SAI1_SD_A,USART2_RX,DFSDM1_DATIN1,SDMMC2_CK,FMC_NWAIT,DCMI_D10,LCD_B2,EVENTOUT)
- net SR_10CTR: now also U1301.68 (PE15,TIM1_BKIN,FMC_D12,LCD_R7,EVENTOUT); no longer U1301.123 (PD7,DFSDM1_DATIN4,SPI1_MOSI,I2S1_SD,DFSDM1_CKIN1,USART2_CK,SPDIF_RX0,SDMMC2_CMD,FMC_NE1,EVENTOUT)
- net SR_10KCTR: now also U1301.65 (PE12,TIM1_CH3N,SPI4_SCK,DFSDM1_DATIN5,SAI2_SCK_B,FMC_D9,LCD_B4,EVENTOUT); no longer U1301.118 (PD4,DFSDM1_CKIN0,USART2_RTS,FMC_NOE,EVENTOUT)
- net SR_1KCTR: now also U1301.67 (PE14,TIM1_CH4,SPI4_MOSI,SAI2_MCLK_B,FMC_D11,LCD_CLK,EVENTOUT); no longer U1301.119 (PD5,USART2_TX,FMC_NWE,EVENTOUT)
- no-connect marks 44 -> 42
Other:
- moved on the sheet: C1305, FB1301

Commit message: PCB layout
Connections:
- no-connect marks 42 -> 44
Changed lines of the file:
@@
 NoConn ~ 2900 6500
 NoConn ~ 14300 6400
+NoConn ~ 14300 2700
+NoConn ~ 2900 1600
 $EndSCHEMATC
