File: hardware/project/ETH1CLCR1/MCU3.sch (KiCad schematic (older format))
At the start: 20 parts, among them J601 20021111-00010T4LF, U601 STM32F413RGT6Tx, U602 24LC08B-E/MS, Y601 NX3225GD-8MHZ-STD-CRA-3

Commit message: Fixed some mistakes in the foorpeints. BOM list ready.
Parts:
- added C609: 1u, Capacitor_SMD:C_0603_1608Metric_Pad1.05x0.95mm_HandSolder, symbol Device:C
- added FB601: 742792031, Inductor_SMD:L_0805_2012Metric_Pad1.15x1.40mm_HandSolder, symbol Device:Ferrite_Bead
- renumbered C609 to C610, C610 to C611, C611 to C612, C612 to C613
Connections:
- net +3.3VF: now also FB601.2; no longer U601.13 (VDDA)
- net DGNDF: now also C609.2
- new net VDDA: C609.1, FB601.1, U601.13 (VDDA)
Changed lines of the file:
@@
 AR Path="/5DF36C25/5E29D787" Ref="#PWR?"  Part="1"
 AR Path="/5E29C232/5E29D787" Ref="#PWR?"  Part="1"
-AR Path="/5DF38F82/5E29D787" Ref="#PWR0606"  Part="1"
-F 0 "#PWR0606" H 7550 6700 50  0001 C CNN
+AR Path="/5DF38F82/5E29D787" Ref="#PWR0608"  Part="1"
+F 0 "#PWR0608" H 7550 6700 50  0001 C CNN
 F 1 "DGNDF" H 7555 6777 50  0000 C CNN
 F 2 "" H 7550 6950 50  0001 C CNN
@@
 	7300 3100 7400 3100
 Wire Wire Line
-	7800 3100 7800 3150
+	7800 2900 7800 3150
 Wire Wire Line
 	7700 3150 7700 3100
-Connection ~ 7700 3100
-Wire Wire Line
-	7700 3100 7800 3100
 Wire Wire Line
 	7600 3150 7600 3100
@@
 AR Path="/5DF36C25/5E29D7AE" Ref="#PWR?"  Part="1"
 AR Path="/5E29C232/5E29D7AE" Ref="#PWR?"  Part="1"
-AR Path="/5DF38F82/5E29D7AE" Ref="#PWR0613"  Part="1"
-F 0 "#PWR0613" H 13300 6400 50  0001 C CNN
+AR Path="/5DF38F82/5E29D7AE" Ref="#PWR0615"  Part="1"
+F 0 "#PWR0615" H 13300 6400 50  0001 C CNN
 F 1 "DGNDF" H 13305 6477 50  0000 C CNN
 F 2 "" H 13300 6650 50  0001 C CNN
@@
 AR Path="/5DF35BC8/5E74C1B5" Ref="#PWR?"  Part="1"
 AR Path="/5E29C232/5E74C1B5" Ref="#PWR?"  Part="1"
-AR Path="/5DF38F82/5E74C1B5" Ref="#PWR0612"  Part="1"
-F 0 "#PWR0612" H 10000 10350 50  0001 C CNN
+AR Path="/5DF38F82/5E74C1B5" Ref="#PWR0614"  Part="1"
+F 0 "#PWR0614" H 10000 10350 50  0001 C CNN
 F 1 "DGNDF" H 10005 10427 50  0000 C CNN
 F 2 "" H 10000 10600 50  0001 C CNN
@@
 AR Path="/5DCED281/5E7594BE" Ref="C?"  Part="1"
 AR Path="/5E29C232/5E7594BE" Ref="C?"  Part="1"
-AR Path="/5DF38F82/5E7594BE" Ref="C611"  Part="1"
-F 0 "C611" H 15115 5596 50  0000 L CNN
+AR Path="/5DF38F82/5E7594BE" Ref="C612"  Part="1"
+F 0 "C612" H 15115 5596 50  0000 L CNN
 F 1 "8p" H 15115 5505 50  0000 L CNN
 F 2 "Capacitor_SMD:C_0603_1608Metric_Pad1.05x0.95mm_HandSolder" H 15038 5400 50  0001 C CNN
@@
 AR Path="/5DCED281/5E7594C4" Ref="C?"  Part="1"
 AR Path="/5E29C232/5E7594C4" Ref="C?"  Part="1"
-AR Path="/5DF38F82/5E7594C4" Ref="C612"  Part="1"
-F 0 "C612" H 15615 5596 50  0000 L CNN
+AR Path="/5DF38F82/5E7594C4" Ref="C613"  Part="1"
+F 0 "C613" H 15615 5596 50  0000 L CNN
 F 1 "8p" H 15615 5505 50  0000 L CNN
 F 2 "Capacitor_SMD:C_0603_1608Metric_Pad1.05x0.95mm_HandSolder" H 15538 5400 50  0001 C CNN
@@
 Connection ~ 9300 9800
 $Comp
-L ETH1CLCR1:DGNDF #PWR0609
+L ETH1CLCR1:DGNDF #PWR0611
 U 1 1 5E77122F
 P 8000 10600
-F 0 "#PWR0609" H 8000 10350 50  0001 C CNN
+F 0 "#PWR0611" H 8000 10350 50  0001 C CNN
 F 1 "DGNDF" H 8005 10427 50  0000 C CNN
 F 2 "" H 8000 10600 50  0001 C CNN
@@
 $EndComp
 $Comp
-L ETH1CLCR1:DGNDF #PWR0607
+L ETH1CLCR1:DGNDF #PWR0609
 U 1 1 5E7714DB
 P 7550 10600
-F 0 "#PWR0607" H 7550 10350 50  0001 C CNN
+F 0 "#PWR0609" H 7550 10350 50  0001 C CNN
 F 1 "DGNDF" H 7555 10427 50  0000 C CNN
 F 2 "" H 7550 10600 50  0001 C CNN
@@
 	8000 9950 8000 10000
 $Comp
-L Device:C C609
+L Device:C C610
 U 1 1 5E776A2B
 P 13400 5650
-F 0 "C609" V 13148 5650 50  0000 C CNN
+F 0 "C610" V 13148 5650 50  0000 C CNN
 F 1 "2u2" V 13239 5650 50  0000 C CNN
 F 2 "Capacitor_SMD:C_0805_2012Metric_Pad1.15x1.40mm_HandSolder" H 13438 5500 50  0001 C CNN
@@
 	13250 5650 13200 5650
 $Comp
-L ETH1CLCR1:DGNDF #PWR0617
+L ETH1CLCR1:DGNDF #PWR0619
 U 1 1 5E77E2A8
 P 15250 5800
-F 0 "#PWR0617" H 15250 5550 50  0001 C CNN
+F 0 "#PWR0619" H 15250 5550 50  0001 C CNN
 F 1 "DGNDF" H 15255 5627 50  0000 C CNN
 F 2 "" H 15250 5800 50  0001 C CNN
@@
 $EndComp
 $Comp
-L ETH1CLCR1:DGNDF #PWR0614
+L ETH1CLCR1:DGNDF #PWR0616
 U 1 1 5E77E4B3
 P 13600 5650
-F 0 "#PWR0614" H 13600 5400 50  0001 C CNN
+F 0 "#PWR0616" H 13600 5400 50  0001 C CNN
 F 1 "DGNDF" V 13605 5522 50  0000 R CNN
 F 2 "" H 13600 5650 50  0001 C CNN
@@
 	13650 5050 13650 5350
 $Comp
-L Device:C C610
+L Device:C C611
 U 1 1 5E7B49DC
 P 14150 6150
-F 0 "C610" H 14265 6196 50  0000 L CNN
+F 0 "C611" H 14265 6196 50  0000 L CNN
 F 1 "100n" H 14265 6105 50  0000 L CNN
 F 2 "Capacitor_SMD:C_0603_1608Metric_Pad1.05x0.95mm_HandSolder" H 14188 6000 50  0001 C CNN
@@
 AR Path="/5DF36C25/5E7BFF4D" Ref="#PWR?"  Part="1"
 AR Path="/5E29C232/5E7BFF4D" Ref="#PWR?"  Part="1"
-AR Path="/5DF38F82/5E7BFF4D" Ref="#PWR0616"  Part="1"
-F 0 "#PWR0616" H 14150 6050 50  0001 C CNN
+AR Path="/5DF38F82/5E7BFF4D" Ref="#PWR0618"  Part="1"
+F 0 "#PWR0618" H 14150 6050 50  0001 C CNN
 F 1 "DGNDF" H 14155 6127 50  0000 C CNN
 F 2 "" H 14150 6300 50  0001 C CNN
@@
 $EndComp
 $Comp
-L ETH1CLCR1:+3.3VF #PWR0608
+L ETH1CLCR1:+3.3VF #PWR0610
 U 1 1 5E94791E
 P 8000 9950
-F 0 "#PWR0608" H 8000 9800 50  0001 C CNN
+F 0 "#PWR0610" H 8000 9800 50  0001 C CNN
 F 1 "+3.3VF" H 8015 10123 50  0000 C CNN
 F 2 "" H 8000 9950 50  0001 C CNN
@@
 $EndComp
 $Comp
-L ETH1CLCR1:+3.3VF #PWR0610
+L ETH1CLCR1:+3.3VF #PWR0612
 U 1 1 5E949139
 P 9300 9750
-F 0 "#PWR0610" H 9300 9600 50  0001 C CNN
+F 0 "#PWR0612" H 9300 9600 50  0001 C CNN
 F 1 "+3.3VF" H 9315 9923 50  0000 C CNN
 F 2 "" H 9300 9750 50  0001 C CNN
@@
 $EndComp
 $Comp
-L ETH1CLCR1:+3.3VF #PWR0611
+L ETH1CLCR1:+3.3VF #PWR0613
 U 1 1 5E9493FF
 P 10000 10050
-F 0 "#PWR0611" H 10000 9900 50  0001 C CNN
+F 0 "#PWR0613" H 10000 9900 50  0001 C CNN
 F 1 "+3.3VF" H 10015 10223 50  0000 C CNN
 F 2 "" H 10000 10050 50  0001 C CNN
@@
 $EndComp
 $Comp
-L ETH1CLCR1:+3.3VF #PWR0615
+L ETH1CLCR1:+3.3VF #PWR0617
 U 1 1 5E9495AA
 P 14150 5600
-F 0 "#PWR0615" H 14150 5450 50  0001 C CNN
+F 0 "#PWR0617" H 14150 5450 50  0001 C CNN
 F 1 "+3.3VF" H 14165 5773 50  0000 C CNN
 F 2 "" H 14150 5600 50  0001 C CNN
@@
 $EndComp
 $Comp
-L ETH1CLCR1:+3.3VF #PWR0605
+L ETH1CLCR1:+3.3VF #PWR0607
 U 1 1 5E94B0CB
 P 7550 3050
-F 0 "#PWR0605" H 7550 2900 50  0001 C CNN
+F 0 "#PWR0607" H 7550 2900 50  0001 C CNN
 F 1 "+3.3VF" H 7565 3223 50  0000 C CNN
 F 2 "" H 7550 3050 50  0001 C CNN
@@
 Wire Wire Line
 	1950 10700 2450 10700
+$Comp
+L Device:Ferrite_Bead FB?
+U 1 1 5E2F3822
+P 5700 10300
+AR Path="/5DCED281/5E2F3822" Ref="FB?"  Part="1"
+AR Path="/5DF35BC8/5E2F3822" Ref="FB?"  Part="1"
+AR Path="/5DEACD0F/5E2F3822" Ref="FB?"  Part="1"
+AR Path="/5DF38F82/5E2F3822" Ref="FB601"  Part="1"
+F 0 "FB601" V 5426 10300 50  0000 C CNN
+F 1 "742792031" V 5517 10300 50  0000 C CNN
+F 2 "Inductor_SMD:L_0805_2012Metric_Pad1.15x1.40mm_HandSolder" V 5630 10300 50  0001 C CNN
+F 3 "~" H 5700 10300 50  0001 C CNN
+	1    5700 10300
+	0    -1   1    0
+$EndComp
+$Comp
+L Device:C C?
+U 1 1 5E2F3828
+P 5450 10500
+AR Path="/5DCED281/5E2F3828" Ref="C?"  Part="1"
+AR Path="/5DF35BC8/5E2F3828" Ref="C?"  Part="1"
+AR Path="/5DEACD0F/5E2F3828" Ref="C?"  Part="1"
+AR Path="/5DF38F82/5E2F3828" Ref="C609"  Part="1"
+F 0 "C609" H 5565 10546 50  0000 L CNN
+F 1 "1u" H 5565 10455 50  0000 L CNN
+F 2 "Capacitor_SMD:C_0603_1608Metric_Pad1.05x0.95mm_HandSolder" H 5488 10350 50  0001 C CNN
+F 3 "~" H 5450 10500 50  0001 C CNN
+	1    5450 10500
+	-1   0    0    -1
+$EndComp
+Wire Wire Line
+	5550 10300 5450 10300
+Wire Wire Line
+	5450 10300 5450 10350
+Wire Wire Line
+	5450 10700 5450 10650
+Wire Wire Line
+	5450 10300 5150 10300
+Connection ~ 5450 10300
+$Comp
+L ETH1CLCR1:DGNDF #PWR?
+U 1 1 5E2F3834
+P 5450 10700
+AR Path="/5DEACD0F/5E2F3834" Ref="#PWR?"  Part="1"
+AR Path="/5DF38F82/5E2F3834" Ref="#PWR0605"  Part="1"
+F 0 "#PWR0605" H 5450 10450 50  0001 C CNN
+F 1 "DGNDF" H 5455 10527 50  0000 C CNN
+F 2 "" H 5450 10700 50  0001 C CNN
+F 3 "" H 5450 10700 50  0001 C CNN
+	1    5450 10700
+	-1   0    0    -1
+$EndComp
+$Comp
+L ETH1CLCR1:+3.3VF #PWR0606
+U 1 1 5E3103B6
+P 6150 10200
+F 0 "#PWR0606" H 6150 10050 50  0001 C CNN
+F 1 "+3.3VF" H 6165 10373 50  0000 C CNN
+F 2 "" H 6150 10200 50  0001 C CNN
+F 3 "" H 6150 10200 50  0001 C CNN
+	1    6150 10200
+	1    0    0    -1
+$EndComp
+Wire Wire Line
+	6150 10200 6150 10300
+Wire Wire Line
+	5850 10300 6150 10300
+Text Label 7800 2900 3    50   ~ 0
+VDDA
+Text Label 5150 10300 0    50   ~ 0
+VDDA
 $EndSCHEMATC

Commit message: PCB layout
Connections:
- net ANALOG_SWITCH: now also U601.40 (PC9,MCO_2,TIM3_CH4,TIM8_CH4,I2C3_SDA,I2S2_CKIN,DFSDM2_DATIN3,QUADSPI_BK1_IO0,SDIO_D1,EVENTOUT); no longer U601.37 (PC6,TIM3_CH1,TIM8_CH1,I2CFMP1_SCL,I2S2_MCK,DFSDM1_CKIN3,DFSDM2_DATIN6,USART6_TX,FSMC_D1,FSMC_DA1,SDIO_D6,EVENTOUT)
- net DDS_DAC_RSTSEL: now also U601.41 (PA8,MCO_1,TIM1_CH1,I2C3_SCL,DFSDM1_CKOUT,USART1_CK,UART7_RX,USB_FS_SOF,CAN3_RX,SDIO_D1,EVENTOUT); no longer U601.14 (PA0,TIM2_CH1,TIM2_ETR,_TIM5_CH1,TIM8_ETR,USART2_CTS,UART4_TX,EVENTOUT,ADC1_IN0,_WKUP1)
- net DDS_DAC_SCLK: now also U601.26 (PB0,TIM1_CH2N,TIM3_CH3,TIM8_CH2N,SPI5_SCK,I2S5_CK,EVENTOUT,ADC1_IN8); no longer U601.21 (PA5,TIM2_CH1,TIM2_ETR,TIM8_CH1N,SPI1_SCK,I2S1_CK,DFSDM1_CKIN1,FSMC_D7,FSMC_DA7,EVENTOUT,ADC1_IN5,DAC_OUT2)
- net DDS_DAC_SDIN: now also U601.43 (PA10,TIM1_CH3,DFSDM2_DATIN3,SPI2_MOSI,I2S2_SD,SPI5_MOSI,I2S5_SD,USART1_RX,USB_FS_ID,EVENTOUT); no longer U601.23 (PA7,TIM1_CH1N,TIM3_CH2,TIM8_CH1N,SPI1MOSI,I2S1_SD,DFSDM2_DATIN1,TIM14_CH1,QUADSPI_BK2_IO1,EVENTOUT,ADC1_IN7)
- net DDS_DAC_SDO: now also U601.45 (PA12,TIM1_ETR,DFSDM2_DATIN5,SPI2_MISO,SPI5_MISO,USART1_RTS,USART6_RX,CAN1_TX,USB_FS_DP,UART4_TX,EVENTOUT); no longer U601.22 (PA6,TIM1_BKIN,TIM3_CH1,TIM8_BKIN,SPI1_MISO,I2S2_MCK,DFSDM2_CKIN1,TIM13_CH1,QUADSPI_BK2_IO0,SDIO_CMD,EVENTOUT,ADC1_IN6)
- net DDS_DAC_~LDAC: now also U601.28 (PB2,LPTIM1_OUT,DFSDM1_CKIN0,QUADSPI_CLK,EVENTOUT,BOOT1); no longer U601.16 (PA2,TIM2_CH3,_TIM5_CH3,TIM9_CH1,I2S2_CKIN,USART2_TX,FSMC_D4,FSMC_DA4,EVENTOUT,ADC1_IN2)
- net DDS_DAC_~RESET: now also U601.42 (PA9,TIM1_CH2,DFSDM2_CKIN3,I2C3_SMBA,SPI2_SCK,I2S2_CK,USART1_TX,USB_FS_VBUS,SDIO_D2,EVENTOUT); no longer U601.17 (PA3,TIM2_CH4,_TIM5_CH4,TIM9_CH2,I2S2_MCK,USART2_RX,SAI1_SD_B,FSMC_D5,FSMC_DA5,EVENTOUT,ADC1_IN3)
- net DDS_DAC_~SYNC: now also U601.27 (PB1,TIM1_CH3N,TIM3_CH4,TIM8_CH3N,SPI5_NSS,I2S5_WS,DFSDM1_DATIN0,QUADSPI_CLK,EVENTOUT,ADC1_IN9); no longer U601.50 (PA15,JTDI,TIM2_CH1,TIM2_ETR,SPI1_NSS,I2S1_WS,SPI3_NSS,I2S3_WS,USART1_TX,UART7_TX,SAI1_MCLK_A,CAN3_TX,EVENTOUT)
- net DDS_FGEN_FSELECT: now also U601.17 (PA3,TIM2_CH4,_TIM5_CH4,TIM9_CH2,I2S2_MCK,USART2_RX,SAI1_SD_B,FSMC_D5,FSMC_DA5,EVENTOUT,ADC1_IN3); no longer U601.28 (PB2,LPTIM1_OUT,DFSDM1_CKIN0,QUADSPI_CLK,EVENTOUT,BOOT1)
- net DDS_FGEN_PSEL0: now also U601.24 (PC4,DFSDM2_CKIN2,I2S1_MCK,_QUADSPI_BK2_IO2,FSMC_NE4,EVENTOUT,ADC1_IN14); no longer U601.41 (PA8,MCO_1,TIM1_CH1,I2C3_SCL,DFSDM1_CKOUT,USART1_CK,UART7_RX,USB_FS_SOF,CAN3_RX,SDIO_D1,EVENTOUT)
- net DDS_FGEN_PSEL1: now also U601.25 (PC5,DFSDM2_DATIN2,I2CFMP1_SMBA,USART3_RX,QUADSPI_BK2_IO3,FSMC_NOE,EVENTOUT,ADC1_IN15); no longer U601.42 (PA9,TIM1_CH2,DFSDM2_CKIN3,I2C3_SMBA,SPI2_SCK,I2S2_CK,USART1_TX,USB_FS_VBUS,SDIO_D2,EVENTOUT)
- net DDS_FGEN_SCLK: now also U601.21 (PA5,TIM2_CH1,TIM2_ETR,TIM8_CH1N,SPI1_SCK,I2S1_CK,DFSDM1_CKIN1,FSMC_D7,FSMC_DA7,EVENTOUT,ADC1_IN5,DAC_OUT2); no longer U601.26 (PB0,TIM1_CH2N,TIM3_CH3,TIM8_CH2N,SPI5_SCK,I2S5_CK,EVENTOUT,ADC1_IN8)
- net DDS_FGEN_SDATA: now also U601.23 (PA7,TIM1_CH1N,TIM3_CH2,TIM8_CH1N,SPI1MOSI,I2S1_SD,DFSDM2_DATIN1,TIM14_CH1,QUADSPI_BK2_IO1,EVENTOUT,ADC1_IN7); no longer U601.43 (PA10,TIM1_CH3,DFSDM2_DATIN3,SPI2_MOSI,I2S2_SD,SPI5_MOSI,I2S5_SD,USART1_RX,USB_FS_ID,EVENTOUT)
- net DDS_FGEN_~FSYNC: now also U601.20 (PA4,SPI1_NSS,I2S1_WS,SPI3_NSS,I2S3_WS,USART2_CK,DFSDM1_DATIN1,FSMC_D6,FSMC_DA6,EVENTOUT,ADC1_IN4,DAC_OUT1); no longer U601.27 (PB1,TIM1_CH3N,TIM3_CH4,TIM8_CH3N,SPI5_NSS,I2S5_WS,DFSDM1_DATIN0,QUADSPI_CLK,EVENTOUT,ADC1_IN9)
- net DDS_MDAC_DIN: now also U601.36 (PB15,RTC_REFIN,TIM1_CH3N,TIM8_CH3N,I2CFMP1_SCL,_SPI2_MOSI,I2S2_SD,DFSDM1_CKIN2,TIM12_CH2,_SDIO_CK,EVENTOU); no longer U601.15 (PA1,TIM2_CH2,TIM5_CH2,SPI4_MOSI,I2S4_SD,USART2_RTS,UART4_RX,QUADSPI_BK1_IO3,EVENTOUT,ADC1_IN1)
- net MCU3_NSS: now also U601.50 (PA15,JTDI,TIM2_CH1,TIM2_ETR,SPI1_NSS,I2S1_WS,SPI3_NSS,I2S3_WS,USART1_TX,UART7_TX,SAI1_MCLK_A,CAN3_TX,EVENTOUT); no longer U601.20 (PA4,SPI1_NSS,I2S1_WS,SPI3_NSS,I2S3_WS,USART2_CK,DFSDM1_DATIN1,FSMC_D6,FSMC_DA6,EVENTOUT,ADC1_IN4,DAC_OUT1)
Other:
- note added: "SPI1"
- note added: "SPI2"
- note added: "SPI3"
- note added: "SPI5"
Changed lines of the file:
@@
 	1    0    0    -1
 $EndComp
-$Comp
-L ETH1CLCR1:STM32F413RGT6Tx U601
-U 1 1 5DD8B08C
-P 7550 5000
-F 0 "U601" H 2050 6800 50  0000 C CNN
-F 1 "STM32F413RGT6Tx" H 12750 6800 50  0000 C CNN
-F 2 "Package_QFP:LQFP-64_10x10mm_P0.5mm" H 850 4400 50  0001 C CNN
-F 3 "" H 850 4400 50  0001 C CNN
-	1    7550 5000
-	1    0    0    -1
-$EndComp
-Text HLabel 13250 3450 2    50   Output ~ 0
+Text HLabel 1850 3750 0    50   Output ~ 0
 DDS_FGEN_~FSYNC
-Text HLabel 1850 4350 0    50   Output ~ 0
+Text HLabel 1850 4050 0    50   Output ~ 0
 DDS_FGEN_SDATA
-Text HLabel 13250 3350 2    50   Output ~ 0
+Text HLabel 1850 3850 0    50   Output ~ 0
 DDS_FGEN_SCLK
 Wire Wire Line
@@
 Wire Wire Line
 	1850 4350 1900 4350
-NoConn ~ 1900 4550
 Text HLabel 13250 4450 2    50   Output ~ 0
 DDS_MDAC_~SYNC
 Text HLabel 13250 4550 2    50   Output ~ 0
 DDS_MDAC_SCLK
-Text HLabel 1850 3450 0    50   Output ~ 0
+Text HLabel 13250 4750 2    50   Output ~ 0
 DDS_MDAC_DIN
 Wire Wire Line
 	13250 4550 13200 4550
 Wire Wire Line
-	1850 3450 1900 3450
+	1850 5450 1900 5450
 Wire Wire Line
 	13250 4450 13200 4450
 Wire Wire Line
 	13250 3450 13200 3450
-Text HLabel 1850 4850 0    50   Output ~ 0
+Text HLabel 13250 3450 2    50   Output ~ 0
 DDS_DAC_~SYNC
-Text HLabel 1850 3850 0    50   Output ~ 0
+Text HLabel 13250 3350 2    50   Output ~ 0
 DDS_DAC_SCLK
-Text HLabel 1850 4050 0    50   Output ~ 0
-DDS_DAC_SDIN
 Wire Wire Line
 	1850 3850 1900 3850
@@
 Wire Wire Line
 	1900 6050 1850 6050
-Text HLabel 1850 6050 0    50   Input ~ 0
-MCU3_SCLK
-Wire Wire Line
-	1900 3750 1850 3750
-Text HLabel 1850 3750 0    50   Input ~ 0
-MCU3_NSS
+Wire Wire Line
+	1900 4850 1850 4850
+Text HLabel 1850 4250 0    50   Output ~ 0
+DDS_DAC_~RESET
+Text HLabel 13250 3550 2    50   Output ~ 0
+DDS_DAC_~LDAC
+Text HLabel 1850 4150 0    50   Output ~ 0
+DDS_DAC_RSTSEL
+Wire Wire Line
+	1850 3750 1900 3750
+Wire Wire Line
+	1850 3650 1900 3650
+Wire Wire Line
+	1850 5550 1900 5550
+Text HLabel 1850 5450 0    50   Output ~ 0
+DDS_FGEN_PSEL0
+Text HLabel 1850 5550 0    50   Output ~ 0
+DDS_FGEN_PSEL1
+Text HLabel 1850 4550 0    50   Input ~ 0
+DDS_DAC_SDO
 Text HLabel 1850 3650 0    50   Output ~ 0
-DDS_DAC_~RESET
-Text HLabel 1850 3550 0    50   Output ~ 0
-DDS_DAC_~LDAC
-Text HLabel 1850 3350 0    50   Output ~ 0
-DDS_DAC_RSTSEL
-Wire Wire Line
-	1850 4850 1900 4850
-Wire Wire Line
-	1850 3650 1900 3650
-Wire Wire Line
-	1850 3550 1900 3550
-Wire Wire Line
-	1850 3350 1900 3350
-NoConn ~ 1900 4450
-Text HLabel 1850 4150 0    50   Output ~ 0
-DDS_FGEN_PSEL0
-Text HLabel 1850 4250 0    50   Output ~ 0
-DDS_FGEN_PSEL1
-Text HLabel 1850 3950 0    50   Input ~ 0
-DDS_DAC_SDO
-Wire Wire Line
-	1850 3950 1900 3950
-Wire Wire Line
-	1850 4250 1900 4250
-Wire Wire Line
-	1900 4150 1850 4150
-Text HLabel 13250 3550 2    50   Output ~ 0
 DDS_FGEN_FSELECT
 Wire Wire Line
@@
 NoConn ~ 13200 3750
 NoConn ~ 13200 4150
-NoConn ~ 13200 4650
-NoConn ~ 13200 4750
 NoConn ~ 1900 6350
 NoConn ~ 1900 6550
-NoConn ~ 1900 5550
-NoConn ~ 1900 5450
 NoConn ~ 1900 5150
 NoConn ~ 1900 5050
@@
 Wire Wire Line
 	4500 10250 4500 10350
-Text HLabel 1850 5650 0    50   Output ~ 0
+Text HLabel 1850 5950 0    50   Output ~ 0
 ANALOG_SWITCH
 Wire Wire Line
-	1850 5650 1900 5650
+	1850 5950 1900 5950
 $Comp
 L ETH1CLCR1:+3.3VF #PWR0601
@@
 	1    0    0    -1
 $EndComp
-Text HLabel 1850 6150 0    50   Output ~ 0
-MCU3_MISO
-Text HLabel 1850 6250 0    50   Input ~ 0
-MCU3_MOSI
-NoConn ~ 1900 5750
 NoConn ~ 1900 5850
-NoConn ~ 1900 5950
 NoConn ~ 1900 5350
 NoConn ~ 13200 4350
@@
 Text Label 5150 10300 0    50   ~ 0
 VDDA
+Text HLabel 1850 4850 0    50   Input ~ 0
+MCU3_NSS
+Text HLabel 1850 6050 0    50   Input ~ 0
+MCU3_SCLK
+Text HLabel 1850 6150 0    50   Output ~ 0
+MCU3_MISO
+Text HLabel 1850 6250 0    50   Input ~ 0
+MCU3_MOSI
+Text Notes 1100 6200 0    50   ~ 0
+SPI3
+Text Notes 1100 4900 0    50   ~ 0
+SPI3
+NoConn ~ 1900 3950
+Text Notes 900  3950 0    50   ~ 0
+SPI1
+NoConn ~ 1900 3450
+NoConn ~ 1900 3550
+Wire Wire Line
+	13250 4750 13200 4750
+Text Notes 14050 4600 0    50   ~ 0
+SPI2
+Text HLabel 1850 4350 0    50   Output ~ 0
+DDS_DAC_SDIN
+Wire Wire Line
+	1850 4550 1900 4550
+Text Notes 13950 3400 0    50   ~ 0
+SPI5
+Text Notes 1050 4600 0    50   ~ 0
+SPI5
+Text Notes 1000 4350 0    50   ~ 0
+SPI5
+Wire Wire Line
+	1850 4250 1900 4250
+NoConn ~ 1900 5650
+NoConn ~ 1900 3350
+NoConn ~ 1900 4450
+Wire Wire Line
+	1900 4150 1850 4150
+$Comp
+L ETH1CLCR1:STM32F413RGT6Tx U601
+U 1 1 5DD8B08C
+P 7550 5000
+F 0 "U601" H 2050 6800 50  0000 C CNN
+F 1 "STM32F413RGT6Tx" H 12750 6800 50  0000 C CNN
+F 2 "Package_QFP:LQFP-64_10x10mm_P0.5mm" H 850 4400 50  0001 C CNN
+F 3 "" H 850 4400 50  0001 C CNN
+	1    7550 5000
+	1    0    0    -1
+$EndComp
+NoConn ~ 13200 4650
+NoConn ~ 1900 5750
 $EndSCHEMATC

Commit message: PCB layout
Connections:
- net ANALOG_SWITCH: now also U601.29 (PB10,TIM2_CH3,I2C2_SCL,SPI2_SCK,I2S2_CK,I2S3_MCK,USART3_TX,I2CFMP1_SCL,DFSDM2_CKOUT,SDIO_D7,EVENTOUT); no longer U601.40 (PC9,MCO_2,TIM3_CH4,TIM8_CH4,I2C3_SDA,I2S2_CKIN,DFSDM2_DATIN3,QUADSPI_BK1_IO0,SDIO_D1,EVENTOUT)
Changed lines of the file:
@@
 Wire Wire Line
 	4500 10250 4500 10350
-Text HLabel 1850 5950 0    50   Output ~ 0
+Text HLabel 13250 4350 2    50   Output ~ 0
 ANALOG_SWITCH
 Wire Wire Line
-	1850 5950 1900 5950
+	13250 4350 13200 4350
 $Comp
 L ETH1CLCR1:+3.3VF #PWR0601
@@
 NoConn ~ 1900 5850
 NoConn ~ 1900 5350
-NoConn ~ 13200 4350
 NoConn ~ 13200 4250
 $Comp
@@
 NoConn ~ 13200 4650
 NoConn ~ 1900 5750
+NoConn ~ 1900 5950
 $EndSCHEMATC

Commit message: PCB done.
Connections:
- net EEPROM_WP: now also U601.56 (PB4,TRST,TIM3_CH1,SPI1_MISO,SPI3_MISO,I2S3ext_SD,UART7_TX,I2C3_SDA,SAI1_SCK_A,CAN3_TX,SDIO_D0,EVENTOUT); no longer U601.57 (PB5,LPTIM1_IN1,TIM3_CH2,I2C1_SMBA,SPI1_MOSI,I2S1_SD,SPI3_MOSI,I2S3_SD,CAN2_RX,SAI1_FS_A,UART5_RX,SDIO_D3,EVENTOUT)
Other:
- note removed: "SPI1"
- note removed: "SPI2"
- note removed: "SPI3"
- note removed: "SPI5"
- moved on the sheet: C609, FB601, J601, R601, R602, U602
